Commit message: Chassis

File: ros2_ws/src/my_rover/urdf/chassis.xacro (robot description, xacro)
@@ -9,15 +9,15 @@
         <visual>
             <geometry>
-                <box size='${chassis-length} ${chassis-width} ${chassis-height}'/>
+                <box size='${chassis_length} ${chassis_width} ${chassis_height}'/>
             </geometry>
         </visual>
         <collision>
             <geometry>
-                <box size='${chassis-length} ${chassis-width} ${chassis-height}'/>
+                <box size='${chassis_length} ${chassis_width} ${chassis_height}'/>
             </geometry>
         </collision>
         <inertial>
             <mass value='10'/>
-            <xacro:box_inertia m="10" x="${chassis-length}" y="${chassis-width}" z="${chassis-height}"/>
+            <xacro:box_inertia m="10" x="${chassis_length}" y="${chassis_width}" z="${chassis_height}"/>
         </inertial>
     </link>

File: ros2_ws/src/my_rover/urdf/rover_properties.xacro (robot description, xacro)
@@ -1,6 +1,6 @@
 <?xml version="1.0"?>
 <robot xmlns:xacro='http://www.ros.org/wiki/xacro' name='my_rover'>
-    <xacro:property name='chassis-length' value='1.5'/>
-    <xacro:property name='chassis-width' value='1'/>
-    <xacro:property name='chassis-height' value='1'/>
+    <xacro:property name='chassis_length' value='1.5'/>
+    <xacro:property name='chassis_width' value='1'/>
+    <xacro:property name='chassis_height' value='1'/>
 </robot>

Commit message: Chassis

File: ros2_ws/src/my_rover/urdf/chassis.xacro (robot description, xacro)
@@ -11,4 +11,7 @@
                 <box size='${chassis_length} ${chassis_width} ${chassis_height}'/>
             </geometry>
+            <material name='blue'>
+                <color rgba='0.2 0.2 1.0 1.0'/>
+            </material>
         </visual>
         <collision>

Commit message: Chassis

File: ros2_ws/src/my_rover/urdf/chassis.xacro (robot description, xacro)
@@ -8,4 +8,5 @@
     <link name='chassis'>
         <visual>
+            <origin xyz="0 0 0" rpy="0 0 0"/>
             <geometry>
                 <box size='${chassis_length} ${chassis_width} ${chassis_height}'/>
@@ -16,4 +17,5 @@
         </visual>
         <collision>
+            <origin xyz="0 0 0" rpy="0 0 0"/>
             <geometry>
                 <box size='${chassis_length} ${chassis_width} ${chassis_height}'/>
@@ -21,4 +23,5 @@
         </collision>
         <inertial>
+            <origin xyz="0 0 0" rpy="0 0 0"/>
             <mass value='10'/>
             <xacro:box_inertia m="10" x="${chassis_length}" y="${chassis_width}" z="${chassis_height}"/>
