Commit message: Suspension_rods

File: ros2_ws/src/my_rover/urdf/rover.urdf.xacro (robot description, xacro)
@@ -7,4 +7,5 @@
     <xacro:include filename="rover_properties.xacro"/>
     <xacro:include filename="chassis.xacro"/>
+    <xacro:include filename="suspension.xacro"/>
     <xacro:include filename="wheel.xacro"/>
     <link name='world'/>

File: ros2_ws/src/my_rover/urdf/rover_properties.xacro (robot description, xacro)
@@ -4,3 +4,5 @@
     <xacro:property name='chassis_width' value='1'/>
     <xacro:property name='chassis_height' value='0.5'/>
+    <xacro:property name='chassis_suspension_rod_length' value='0.1'/>
+    <xacro:property name='chassis_suspension_rod_radius' value='0.05'/>
 </robot>
