Commit message: Wheels

File: ros2_ws/src/my_rover/urdf/wheel.xacro (robot description, xacro)
@@ -1,3 +1,111 @@
 <?xml version="1.0"?>
 <robot xmlns:xacro="http://www.ros.org/wiki/xacro" name="my_rover">
+    <link name='wheel-base'>
+        <visual>
+            <origin xyz='0 0 0' rpy='0 0 0'/>
+            <geometry>
+                <cylinder radius='${wheel_base_radius}' length='${wheel_base_length}'/>
+                <material name='black'>
+                    <color rgba='0.2 0.2 0.2 1.0'/>
+                </material>
+            </geometry>
+            <collision>
+                <origin xyz='0 0 0' rpy='0 0 0'/>
+                <geometry>
+                    <cylinder radius='${wheel_base_radius}' length='${wheel_base_length}'/>
+                </geometry>
+            </collision>
+            <inertial>
+                <origin xyz='0 0 0' rpy='0 0 0'/>
+                <mass value='1'/>
+                <xacro:cylinder_inertia m="1" r="${wheel_base_radius}" h="${wheel_base_length}"/>
+            </inertial>
+        </visual>
+    </link>
+    <link name='wheel-base_2'>
+        <visual>
+            <origin xyz='0 0 0' rpy='0 0 0'/>
+            <geometry>
+                <cylinder radius='${wheel_base_radius}' length='${wheel_base_length}'/>
+                <material name='black'>
+                    <color rgba='0.2 0.2 0.2 1.0'/>
+                </material>
+            </geometry>
+            <collision>
+                <origin xyz='0 0 0' rpy='0 0 0'/>
+                <geometry>
+                    <cylinder radius='${wheel_base_radius}' length='${wheel_base_length}'/>
+                </geometry>
+            </collision>
+            <inertial>
+                <origin xyz='0 0 0' rpy='0 0 0'/>
+                <mass value='1'/>
+                <xacro:cylinder_inertia m="1" r="${wheel_base_radius}" h="${wheel_base_length}"/>
+            </inertial>
+        </visual>
+    </link>
+    <link name='wheel-base_3'>
+        <visual>
+            <origin xyz='0 0 0' rpy='0 0 0'/>
+            <geometry>
+                <cylinder radius='${wheel_base_radius}' length='${wheel_base_length}'/>
+                <material name='black'>
+                    <color rgba='0.2 0.2 0.2 1.0'/>
+                </material>
+            </geometry>
+            <collision>
+                <origin xyz='0 0 0' rpy='0 0 0'/>
+                <geometry>
+                    <cylinder radius='${wheel_base_radius}' length='${wheel_base_length}'/>
+                </geometry>
+            </collision>
+            <inertial>
+                <origin xyz='0 0 0' rpy='0 0 0'/>
+                <mass value='1'/>
+                <xacro:cylinder_inertia m="1" r="${wheel_base_radius}" h="${wheel_base_length}"/>
+            </inertial>
+        </visual>
+    </link>
+    <link name='wheel-base_4'>
+        <visual>
+            <origin xyz='0 0 0' rpy='0 0 0'/>
+            <geometry>
+                <cylinder radius='${wheel_base_radius}' length='${wheel_base_length}'/>
+                <material name='black'>
+                    <color rgba='0.2 0.2 0.2 1.0'/>
+                </material>
+            </geometry>
+            <collision>
+                <origin xyz='0 0 0' rpy='0 0 0'/>
+                <geometry>
+                    <cylinder radius='${wheel_base_radius}' length='${wheel_base_length}'/>
+                </geometry>
+            </collision>
+            <inertial>
+                <origin xyz='0 0 0' rpy='0 0 0'/>
+                <mass value='1'/>
+                <xacro:cylinder_inertia m="1" r="${wheel_base_radius}" h="${wheel_base_length}"/>
+            </inertial>
+        </visual>
+    </link>
+    <joint name='wheel_base_joint' type='fixed'>
+        <parent link='suspension_rod'/>
+        <child link='wheel-base'/>
+        <origin xyz='${suspension_rod_length/2} 0 0' rpy='0 0 0'/>
+    </joint>
+    <joint name='wheel_base_2_joint' type='fixed'>
+        <parent link='suspension_rod_2'/>
+        <child link='wheel-base_2'/>
+        <origin xyz='${suspension_rod_length/2} 0 0' rpy='0 0 0'/>
+    </joint>
+    <joint name='wheel_base_3_joint' type='fixed'>
+        <parent link='suspension_rod_3'/>
+        <child link='wheel-base_3'/>
+        <origin xyz='${suspension_rod_length/2} 0 0' rpy='0 0 0'/>
+    </joint>
+    <joint name='wheel_base_4_joint' type='fixed'>
+        <parent link='suspension_rod_4'/>
+        <child link='wheel-base_4'/>
+        <origin xyz='${suspension_rod_length/2} 0 0' rpy='0 0 0'/>
+    </joint>
 </robot>

Commit message: Wheels

File: ros2_ws/src/my_rover/urdf/wheel.xacro (robot description, xacro)
@@ -92,20 +92,20 @@
         <parent link='suspension_rod'/>
         <child link='wheel-base'/>
-        <origin xyz='${suspension_rod_length/2} 0 0' rpy='0 0 0'/>
+        <origin xyz='0 0 ${suspension_rod_length}' rpy='0 0 0'/>
     </joint>
     <joint name='wheel_base_2_joint' type='fixed'>
         <parent link='suspension_rod_2'/>
         <child link='wheel-base_2'/>
-        <origin xyz='${suspension_rod_length/2} 0 0' rpy='0 0 0'/>
+        <origin xyz='0 0 ${suspension_rod_length}' rpy='0 0 0'/>
     </joint>
     <joint name='wheel_base_3_joint' type='fixed'>
         <parent link='suspension_rod_3'/>
         <child link='wheel-base_3'/>
-        <origin xyz='${suspension_rod_length/2} 0 0' rpy='0 0 0'/>
+        <origin xyz='0 0 ${suspension_rod_length}' rpy='0 0 0'/>
     </joint>
     <joint name='wheel_base_4_joint' type='fixed'>
         <parent link='suspension_rod_4'/>
         <child link='wheel-base_4'/>
-        <origin xyz='${suspension_rod_length/2} 0 0' rpy='0 0 0'/>
+        <origin xyz='0 0 ${suspension_rod_length}' rpy='0 0 0'/>
     </joint>
 </robot>

Commit message: Wheels

File: ros2_ws/src/my_rover/urdf/wheel.xacro (robot description, xacro)
@@ -92,5 +92,5 @@
         <parent link='suspension_rod'/>
         <child link='wheel-base'/>
-        <origin xyz='0 0 ${suspension_rod_length}' rpy='0 0 0'/>
+        <origin xyz='0 0 ${suspension_rod_length}' rpy='${pi/2 - atan2(chassis_height/2 ,chassis_length/2)} 0 0'/>
     </joint>
     <joint name='wheel_base_2_joint' type='fixed'>

Commit message: Wheels

File: ros2_ws/src/my_rover/urdf/wheel.xacro (robot description, xacro)
@@ -3,5 +3,5 @@
     <link name='wheel-base'>
         <visual>
-            <origin xyz='0 0 ${wheel_base_length/2}' rpy='0 0 0'/>
+            <origin xyz='0 0 ${-wheel_base_length/2}' rpy='0 0 0'/>
             <geometry>
                 <cylinder radius='${wheel_base_radius}' length='${wheel_base_length}'/>
@@ -12,5 +12,5 @@
         </visual>
         <collision>
-            <origin xyz='0 0 ${wheel_base_length/2}' rpy='0 0 0'/>
+            <origin xyz='0 0 ${-wheel_base_length/2}' rpy='0 0 0'/>
             <geometry>
                 <cylinder radius='${wheel_base_radius}' length='${wheel_base_length}'/>
@@ -18,5 +18,5 @@
         </collision>
         <inertial>
-            <origin xyz='0 0 ${wheel_base_length/2}' rpy='0 0 0'/>
+            <origin xyz='0 0 ${-wheel_base_length/2}' rpy='0 0 0'/>
             <mass value='1'/>
             <xacro:cylinder_inertia m="1" r="${wheel_base_radius}" h="${wheel_base_length}"/>
@@ -25,5 +25,5 @@
     <link name='wheel-base_2'>
         <visual>
-            <origin xyz='0 0 ${wheel_base_length/2}' rpy='0 0 0'/>
+            <origin xyz='0 0 ${-wheel_base_length/2}' rpy='0 0 0'/>
             <geometry>
                 <cylinder radius='${wheel_base_radius}' length='${wheel_base_length}'/>
@@ -34,5 +34,5 @@
         </visual>
         <collision>
-            <origin xyz='0 0 ${wheel_base_length/2}' rpy='0 0 0'/>
+            <origin xyz='0 0 ${-wheel_base_length/2}' rpy='0 0 0'/>
             <geometry>
                 <cylinder radius='${wheel_base_radius}' length='${wheel_base_length}'/>
@@ -40,5 +40,5 @@
         </collision>
         <inertial>
-            <origin xyz='0 0 ${wheel_base_length/2}' rpy='0 0 0'/>
+            <origin xyz='0 0 ${-wheel_base_length/2}' rpy='0 0 0'/>
             <mass value='1'/>
             <xacro:cylinder_inertia m="1" r="${wheel_base_radius}" h="${wheel_base_length}"/>
@@ -47,5 +47,5 @@
     <link name='wheel-base_3'>
         <visual>
-            <origin xyz='0 0 ${wheel_base_length/2}' rpy='0 0 0'/>
+            <origin xyz='0 0 ${-wheel_base_length/2}' rpy='0 0 0'/>
             <geometry>
                 <cylinder radius='${wheel_base_radius}' length='${wheel_base_length}'/>
@@ -56,5 +56,5 @@
         </visual>
         <collision>
-            <origin xyz='0 0 ${wheel_base_length/2}' rpy='0 0 0'/>
+            <origin xyz='0 0 ${-wheel_base_length/2}' rpy='0 0 0'/>
             <geometry>
                 <cylinder radius='${wheel_base_radius}' length='${wheel_base_length}'/>
@@ -62,5 +62,5 @@
         </collision>
         <inertial>
-            <origin xyz='0 0 ${wheel_base_length/2}' rpy='0 0 0'/>
+            <origin xyz='0 0 ${-wheel_base_length/2}' rpy='0 0 0'/>
             <mass value='1'/>
             <xacro:cylinder_inertia m="1" r="${wheel_base_radius}" h="${wheel_base_length}"/>
@@ -69,5 +69,5 @@
     <link name='wheel-base_4'>
         <visual>
-            <origin xyz='0 0 ${wheel_base_length/2}' rpy='0 0 0'/>
+            <origin xyz='0 0 ${-wheel_base_length/2}' rpy='0 0 0'/>
             <geometry>
                 <cylinder radius='${wheel_base_radius}' length='${wheel_base_length}'/>
@@ -78,5 +78,5 @@
         </visual>
         <collision>
-            <origin xyz='0 0 ${wheel_base_length/2}' rpy='0 0 0'/>
+            <origin xyz='0 0 ${-wheel_base_length/2}' rpy='0 0 0'/>
             <geometry>
                 <cylinder radius='${wheel_base_radius}' length='${wheel_base_length}'/>
@@ -84,5 +84,5 @@
         </collision>
         <inertial>
-            <origin xyz='0 0 ${wheel_base_length/2}' rpy='0 0 0'/>
+            <origin xyz='0 0 ${-wheel_base_length/2}' rpy='0 0 0'/>
             <mass value='1'/>
             <xacro:cylinder_inertia m="1" r="${wheel_base_radius}" h="${wheel_base_length}"/>

Commit message: Wheels

File: ros2_ws/src/my_rover/urdf/wheel.xacro (robot description, xacro)
@@ -3,5 +3,5 @@
     <link name='wheel-base'>
         <visual>
-            <origin xyz='0 0 ${-wheel_base_length/2}' rpy='0 0 0'/>
+            <origin xyz='0 0 ${-wheel_base_length/3}' rpy='0 0 0'/>
             <geometry>
                 <cylinder radius='${wheel_base_radius}' length='${wheel_base_length}'/>
@@ -12,5 +12,5 @@
         </visual>
         <collision>
-            <origin xyz='0 0 ${-wheel_base_length/2}' rpy='0 0 0'/>
+            <origin xyz='0 0 ${-wheel_base_length/3}' rpy='0 0 0'/>
             <geometry>
                 <cylinder radius='${wheel_base_radius}' length='${wheel_base_length}'/>
@@ -18,5 +18,5 @@
         </collision>
         <inertial>
-            <origin xyz='0 0 ${-wheel_base_length/2}' rpy='0 0 0'/>
+            <origin xyz='0 0 ${-wheel_base_length/3}' rpy='0 0 0'/>
             <mass value='1'/>
             <xacro:cylinder_inertia m="1" r="${wheel_base_radius}" h="${wheel_base_length}"/>
@@ -25,5 +25,5 @@
     <link name='wheel-base_2'>
         <visual>
-            <origin xyz='0 0 ${-wheel_base_length/2}' rpy='0 0 0'/>
+            <origin xyz='0 0 ${-wheel_base_length/3}' rpy='0 0 0'/>
             <geometry>
                 <cylinder radius='${wheel_base_radius}' length='${wheel_base_length}'/>
@@ -34,5 +34,5 @@
         </visual>
         <collision>
-            <origin xyz='0 0 ${-wheel_base_length/2}' rpy='0 0 0'/>
+            <origin xyz='0 0 ${-wheel_base_length/3}' rpy='0 0 0'/>
             <geometry>
                 <cylinder radius='${wheel_base_radius}' length='${wheel_base_length}'/>
@@ -40,5 +40,5 @@
         </collision>
         <inertial>
-            <origin xyz='0 0 ${-wheel_base_length/2}' rpy='0 0 0'/>
+            <origin xyz='0 0 ${-wheel_base_length/3}' rpy='0 0 0'/>
             <mass value='1'/>
             <xacro:cylinder_inertia m="1" r="${wheel_base_radius}" h="${wheel_base_length}"/>
@@ -47,5 +47,5 @@
     <link name='wheel-base_3'>
         <visual>
-            <origin xyz='0 0 ${-wheel_base_length/2}' rpy='0 0 0'/>
+            <origin xyz='0 0 ${-wheel_base_length/3}' rpy='0 0 0'/>
             <geometry>
                 <cylinder radius='${wheel_base_radius}' length='${wheel_base_length}'/>
@@ -56,5 +56,5 @@
         </visual>
         <collision>
-            <origin xyz='0 0 ${-wheel_base_length/2}' rpy='0 0 0'/>
+            <origin xyz='0 0 ${-wheel_base_length/3}' rpy='0 0 0'/>
             <geometry>
                 <cylinder radius='${wheel_base_radius}' length='${wheel_base_length}'/>
@@ -62,5 +62,5 @@
         </collision>
         <inertial>
-            <origin xyz='0 0 ${-wheel_base_length/2}' rpy='0 0 0'/>
+            <origin xyz='0 0 ${-wheel_base_length/3}' rpy='0 0 0'/>
             <mass value='1'/>
             <xacro:cylinder_inertia m="1" r="${wheel_base_radius}" h="${wheel_base_length}"/>
@@ -69,5 +69,5 @@
     <link name='wheel-base_4'>
         <visual>
-            <origin xyz='0 0 ${-wheel_base_length/2}' rpy='0 0 0'/>
+            <origin xyz='0 0 ${-wheel_base_length/3}' rpy='0 0 0'/>
             <geometry>
                 <cylinder radius='${wheel_base_radius}' length='${wheel_base_length}'/>
@@ -78,5 +78,5 @@
         </visual>
         <collision>
-            <origin xyz='0 0 ${-wheel_base_length/2}' rpy='0 0 0'/>
+            <origin xyz='0 0 ${-wheel_base_length/3}' rpy='0 0 0'/>
             <geometry>
                 <cylinder radius='${wheel_base_radius}' length='${wheel_base_length}'/>
@@ -84,5 +84,5 @@
         </collision>
         <inertial>
-            <origin xyz='0 0 ${-wheel_base_length/2}' rpy='0 0 0'/>
+            <origin xyz='0 0 ${-wheel_base_length/3}' rpy='0 0 0'/>
             <mass value='1'/>
             <xacro:cylinder_inertia m="1" r="${wheel_base_radius}" h="${wheel_base_length}"/>

Commit message: Wheels

File: ros2_ws/src/my_rover/urdf/wheel.xacro (robot description, xacro)
@@ -109,3 +109,119 @@
         <origin xyz='0 0 ${suspension_rod_length}' rpy='${-pi/2 - atan2(chassis_height/2 ,chassis_length/2)} 0 0'/>
     </joint>
+    <link name='wheel_steer'>
+        <visual>
+            <origin xyz='0 0 0' rpy='0 0 0'/>
+            <geometry>
+                <box size='${wheel_steer_length} ${wheel_steer_width} ${wheel_steer_height}'/>
+            </geometry>
+            <material name='gray'>
+                <color rgba='0.5 0.5 0.5 1.0'/>
+            </material>
+        </visual>
+        <collision>
+            <origin xyz='0 0 0' rpy='0 0 0'/>
+            <geometry>
+                <box size='${wheel_steer_length} ${wheel_steer_width} ${wheel_steer_height}'/>
+            </geometry>
+        </collision>
+        <inertial>
+            <origin xyz='0 0 0' rpy='0 0 0'/>
+            <mass value='1'/>
+            <xacro:box_inertia m="1" x="${wheel_steer_length}" y="${wheel_steer_width}" z="${wheel_steer_height}"/>
+        </inertial>
+    </link>
+    <link name='wheel_steer_2'>
+        <visual>
+            <origin xyz='0 0 0' rpy='0 0 0'/>
+            <geometry>
+                <box size='${wheel_steer_length} ${wheel_steer_width} ${wheel_steer_height}'/>
+            </geometry>
+            <material name='gray'>
+                <color rgba='0.5 0.5 0.5 1.0'/>
+            </material>
+        </visual>
+        <collision>
+            <origin xyz='0 0 0' rpy='0 0 0'/>
+            <geometry>
+                <box size='${wheel_steer_length} ${wheel_steer_width} ${wheel_steer_height}'/>
+            </geometry>
+        </collision>
+        <inertial>
+            <origin xyz='0 0 0' rpy='0 0 0'/>
+            <mass value='1'/>
+            <xacro:box_inertia m="1" x="${wheel_steer_length}" y="${wheel_steer_width}" z="${wheel_steer_height}"/>
+        </inertial>
+    </link>
+    <link name='wheel_steer_3'>
+        <visual>
+            <origin xyz='0 0 0' rpy='0 0 0'/>
+            <geometry>
+                <box size='${wheel_steer_length} ${wheel_steer_width} ${wheel_steer_height}'/>
+            </geometry>
+            <material name='gray'>
+                <color rgba='0.5 0.5 0.5 1.0'/>
+            </material>
+        </visual>
+        <collision>
+            <origin xyz='0 0 0' rpy='0 0 0'/>
+            <geometry>
+                <box size='${wheel_steer_length} ${wheel_steer_width} ${wheel_steer_height}'/>
+            </geometry>
+        </collision>
+        <inertial>
+            <origin xyz='0 0 0' rpy='0 0 0'/>
+            <mass value='1'/>
+            <xacro:box_inertia m="1" x="${wheel_steer_length}" y="${wheel_steer_width}" z="${wheel_steer_height}"/>
+        </inertial>
+    </link>
+    <link name='wheel_steer_4'>
+        <visual>
+            <origin xyz='0 0 0' rpy='0 0 0'/>
+            <geometry>
+                <box size='${wheel_steer_length} ${wheel_steer_width} ${wheel_steer_height}'/>
+            </geometry>
+            <material name='gray'>
+                <color rgba='0.5 0.5 0.5 1.0'/>
+            </material>
+        </visual>
+        <collision>
+            <origin xyz='0 0 0' rpy='0 0 0'/>
+            <geometry>
+                <box size='${wheel_steer_length} ${wheel_steer_width} ${wheel_steer_height}'/>
+            </geometry>
+        </collision>
+        <inertial>
+            <origin xyz='0 0 0' rpy='0 0 0'/>
+            <mass value='1'/>
+            <xacro:box_inertia m="1" x="${wheel_steer_length}" y="${wheel_steer_width}" z="${wheel_steer_height}"/>
+        </inertial>
+    </link>
+    <joint name='wheel_steer_joint_1' type='revolute'>
+        <parent link='wheel-base'/>
+        <child link='wheel_steer'/>
+        <origin xyz='0 0 ${-wheel_base_length/3}' rpy='0 0 0'/>
+        <axis xyz='0 0 1'/>
+        <limit lower='-1.57' upper='1.57' effort='1000' velocity='1'/>
+    </joint>
+    <joint name='wheel_steer_joint_2' type='revolute'>
+        <parent link='wheel-base'/>
+        <child link='wheel_steer_2'/>
+        <origin xyz='0 0 ${-wheel_base_length/3}' rpy='0 0 0'/>
+        <axis xyz='0 0 1'/>
+        <limit lower='-1.57' upper='1.57' effort='1000' velocity='1'/>
+    </joint>
+    <joint name='wheel_steer_joint_3' type='revolute'>
+        <parent link='wheel-base'/>
+        <child link='wheel_steer_3'/>
+        <origin xyz='0 0 ${-wheel_base_length/3}' rpy='0 0 0'/>
+        <axis xyz='0 0 1'/>
+        <limit lower='-1.57' upper='1.57' effort='1000' velocity='1'/>
+    </joint>
+    <joint name='wheel_steer_joint_4' type='revolute'>
+        <parent link='wheel-base'/>
+        <child link='wheel_steer_4'/>
+        <origin xyz='0 0 ${-wheel_base_length/3}' rpy='0 0 0'/>
+        <axis xyz='0 0 1'/>
+        <limit lower='-1.57' upper='1.57' effort='1000' velocity='1'/>
+    </joint>
 </robot>

Commit message: Wheels

File: ros2_ws/src/my_rover/urdf/wheel.xacro (robot description, xacro)
@@ -200,10 +200,10 @@
         <parent link='wheel-base'/>
         <child link='wheel_steer'/>
-        <origin xyz='0 0 ${-wheel_base_length/3}' rpy='0 0 0'/>
+        <origin xyz='0 0 ${-wheel_base_length}' rpy='0 0 0'/>
         <axis xyz='0 0 1'/>
         <limit lower='-1.57' upper='1.57' effort='1000' velocity='1'/>
     </joint>
     <joint name='wheel_steer_joint_2' type='revolute'>
-        <parent link='wheel-base'/>
+        <parent link='wheel-base_2'/>
         <child link='wheel_steer_2'/>
         <origin xyz='0 0 ${-wheel_base_length/3}' rpy='0 0 0'/>
@@ -212,5 +212,5 @@
     </joint>
     <joint name='wheel_steer_joint_3' type='revolute'>
-        <parent link='wheel-base'/>
+        <parent link='wheel-base_3'/>
         <child link='wheel_steer_3'/>
         <origin xyz='0 0 ${-wheel_base_length/3}' rpy='0 0 0'/>
@@ -219,5 +219,5 @@
     </joint>
     <joint name='wheel_steer_joint_4' type='revolute'>
-        <parent link='wheel-base'/>
+        <parent link='wheel-base_4'/>
         <child link='wheel_steer_4'/>
         <origin xyz='0 0 ${-wheel_base_length/3}' rpy='0 0 0'/>

Commit message: Wheels

File: ros2_ws/src/my_rover/urdf/wheel.xacro (robot description, xacro)
@@ -200,5 +200,5 @@
         <parent link='wheel-base'/>
         <child link='wheel_steer'/>
-        <origin xyz='0 0 ${-wheel_base_length}' rpy='0 0 0'/>
+        <origin xyz='0 0 ${-wheel_base_length/2 - wheel_steer_height/2}' rpy='0 0 0'/>
         <axis xyz='0 0 1'/>
         <limit lower='-1.57' upper='1.57' effort='1000' velocity='1'/>

Commit message: Wheels

File: ros2_ws/src/my_rover/urdf/wheel.xacro (robot description, xacro)
@@ -200,5 +200,5 @@
         <parent link='wheel-base'/>
         <child link='wheel_steer'/>
-        <origin xyz='0 0 ${-wheel_base_length/2 - wheel_steer_height/2}' rpy='0 0 0'/>
+        <origin xyz='0 0 ${-wheel_base_length - wheel_steer_height/2}' rpy='0 0 0'/>
         <axis xyz='0 0 1'/>
         <limit lower='-1.57' upper='1.57' effort='1000' velocity='1'/>

Commit message: Wheels

File: ros2_ws/src/my_rover/urdf/wheel.xacro (robot description, xacro)
@@ -200,5 +200,5 @@
         <parent link='wheel-base'/>
         <child link='wheel_steer'/>
-        <origin xyz='0 0 ${-wheel_base_length - wheel_steer_height/2}' rpy='0 0 0'/>
+        <origin xyz='0 0 ${-2*wheel_base_length/3 - wheel_steer_height/2}' rpy='0 0 0'/>
         <axis xyz='0 0 1'/>
         <limit lower='-1.57' upper='1.57' effort='1000' velocity='1'/>
