Commit message: Wheels

File: ros2_ws/src/my_rover/urdf/wheel.xacro (robot description, xacro)
@@ -229,17 +229,17 @@
             <origin xyz='0 0 0' rpy='0 0 0'/>
             <geometry>
-                <box size='${wheel_steer_to_wheel_length} ${wheel_steer_to_width} ${wheel_steer_to_height}'/>
-            </geometry>
-        </visual>
-        <collision>
-            <origin xyz='0 0 0' rpy='0 0 0'/>
-            <geometry>
-                <box size='${wheel_steer_to_wheel_length} ${wheel_steer_to_width} ${wheel_steer_to_height}'/>
-            </geometry>
-        </collision>
-        <inertial>
-            <origin xyz='0 0 0' rpy='0 0 0'/>
-            <mass value='1'/>
-            <xacro:box_inertia m="1" x="${wheel_steer_to_wheel_length}" y="${wheel_steer_to_width}" z="${wheel_steer_to_height}"/>
+                <box size='${wheel_steer_to_wheel_length} ${wheel_steer_to_wheel_width} ${wheel_steer_to_wheel_height}'/>
+            </geometry>
+        </visual>
+        <collision>
+            <origin xyz='0 0 0' rpy='0 0 0'/>
+            <geometry>
+                <box size='${wheel_steer_to_wheel_length} ${wheel_steer_to_wheel_width} ${wheel_steer_to_wheel_height}'/>
+            </geometry>
+        </collision>
+        <inertial>
+            <origin xyz='0 0 0' rpy='0 0 0'/>
+            <mass value='1'/>
+            <xacro:box_inertia m="1" x="${wheel_steer_to_wheel_length}" y="${wheel_steer_to_wheel_width}" z="${wheel_steer_to_wheel_height}"/>
         </inertial>
     </link>
@@ -248,17 +248,17 @@
             <origin xyz='0 0 0' rpy='0 0 0'/>
             <geometry>
-                <box size='${wheel_steer_to_wheel_length} ${wheel_steer_to_width} ${wheel_steer_to_height}'/>
-            </geometry>
-        </visual>
-        <collision>
-            <origin xyz='0 0 0' rpy='0 0 0'/>
-            <geometry>
-                <box size='${wheel_steer_to_wheel_length} ${wheel_steer_to_width} ${wheel_steer_to_height}'/>
-            </geometry>
-        </collision>
-        <inertial>
-            <origin xyz='0 0 0' rpy='0 0 0'/>
-            <mass value='1'/>
-            <xacro:box_inertia m="1" x="${wheel_steer_to_wheel_length}" y="${wheel_steer_to_width}" z="${wheel_steer_to_height}"/>
+                <box size='${wheel_steer_to_wheel_length} ${wheel_steer_to_wheel_width} ${wheel_steer_to_wheel_height}'/>
+            </geometry>
+        </visual>
+        <collision>
+            <origin xyz='0 0 0' rpy='0 0 0'/>
+            <geometry>
+                <box size='${wheel_steer_to_wheel_length} ${wheel_steer_to_wheel_width} ${wheel_steer_to_wheel_height}'/>
+            </geometry>
+        </collision>
+        <inertial>
+            <origin xyz='0 0 0' rpy='0 0 0'/>
+            <mass value='1'/>
+            <xacro:box_inertia m="1" x="${wheel_steer_to_wheel_length}" y="${wheel_steer_to_wheel_width}" z="${wheel_steer_to_wheel_height}"/>
         </inertial>
     </link>
@@ -267,17 +267,17 @@
             <origin xyz='0 0 0' rpy='0 0 0'/>
             <geometry>
-                <box size='${wheel_steer_to_wheel_length} ${wheel_steer_to_width} ${wheel_steer_to_height}'/>
-            </geometry>
-        </visual>
-        <collision>
-            <origin xyz='0 0 0' rpy='0 0 0'/>
-            <geometry>
-                <box size='${wheel_steer_to_wheel_length} ${wheel_steer_to_width} ${wheel_steer_to_height}'/>
-            </geometry>
-        </collision>
-        <inertial>
-            <origin xyz='0 0 0' rpy='0 0 0'/>
-            <mass value='1'/>
-            <xacro:box_inertia m="1" x="${wheel_steer_to_wheel_length}" y="${wheel_steer_to_width}" z="${wheel_steer_to_height}"/>
+                <box size='${wheel_steer_to_wheel_length} ${wheel_steer_to_wheel_width} ${wheel_steer_to_wheel_height}'/>
+            </geometry>
+        </visual>
+        <collision>
+            <origin xyz='0 0 0' rpy='0 0 0'/>
+            <geometry>
+                <box size='${wheel_steer_to_wheel_length} ${wheel_steer_to_wheel_width} ${wheel_steer_to_wheel_height}'/>
+            </geometry>
+        </collision>
+        <inertial>
+            <origin xyz='0 0 0' rpy='0 0 0'/>
+            <mass value='1'/>
+            <xacro:box_inertia m="1" x="${wheel_steer_to_wheel_length}" y="${wheel_steer_to_wheel_width}" z="${wheel_steer_to_wheel_height}"/>
         </inertial>
     </link>
@@ -286,11 +286,11 @@
             <origin xyz='0 0 0' rpy='0 0 0'/>
             <geometry>
-                <box size='${wheel_steer_to_wheel_length} ${wheel_steer_to_width} ${wheel_steer_to_height}'/>
-            </geometry>
-        </visual>
-        <collision>
-            <origin xyz='0 0 0' rpy='0 0 0'/>
-            <geometry>
-                <box size='${wheel_steer_to_wheel_length} ${wheel_steer_to_width} ${wheel_steer_to_height}'/>
+                <box size='${wheel_steer_to_wheel_length} ${wheel_steer_to_wheel_width} ${wheel_steer_to_wheel_height}'/>
+            </geometry>
+        </visual>
+        <collision>
+            <origin xyz='0 0 0' rpy='0 0 0'/>
+            <geometry>
+                <box size='${wheel_steer_to_wheel_length} ${wheel_steer_to_wheel_width} ${wheel_steer_to_wheel_height}'/>
             </geometry>
         </collision>

Commit message: Wheels

File: ros2_ws/src/my_rover/urdf/wheel.xacro (robot description, xacro)
@@ -309,5 +309,5 @@
         <parent link='wheel_steer_2'/>
         <child link='wheel_steer_to_wheel_2'/>
-        <origin xyz='${wheel_steer_to_wheel_length/2-wheel_steer_length/2} 0 ${-wheel_steer_to_wheel_height/2-wheel_steer_height/2}' rpy='0 0 0'/>
+        <origin xyz='${-wheel_steer_to_wheel_length/2+wheel_steer_length/2} 0 ${-wheel_steer_to_wheel_height/2-wheel_steer_height/2}' rpy='0 0 0'/>
     </joint>
     <joint name='wheel_steer_to_wheel_joint_3' type='fixed'>
@@ -319,5 +319,5 @@
         <parent link='wheel_steer_4'/>
         <child link='wheel_steer_to_wheel_4'/>
-        <origin xyz='${wheel_steer_to_wheel_length/2-wheel_steer_length/2} 0 ${-wheel_steer_to_wheel_height/2-wheel_steer_height/2}' rpy='0 0 0'/>
+        <origin xyz='${-wheel_steer_to_wheel_length/2+wheel_steer_length/2} 0 ${-wheel_steer_to_wheel_height/2-wheel_steer_height/2}' rpy='0 0 0'/>
     </joint>
 </robot>

Commit message: Wheels

File: ros2_ws/src/my_rover/urdf/wheel.xacro (robot description, xacro)
@@ -314,10 +314,10 @@
         <parent link='wheel_steer_3'/>
         <child link='wheel_steer_to_wheel_3'/>
-        <origin xyz='${wheel_steer_to_wheel_length/2-wheel_steer_length/2} 0 ${-wheel_steer_to_wheel_height/2-wheel_steer_height/2}' rpy='0 0 0'/>
+        <origin xyz='${-wheel_steer_to_wheel_length/2+wheel_steer_length/2} 0 ${-wheel_steer_to_wheel_height/2-wheel_steer_height/2}' rpy='0 0 0'/>
     </joint>
     <joint name='wheel_steer_to_wheel_joint_4' type='fixed'>
         <parent link='wheel_steer_4'/>
         <child link='wheel_steer_to_wheel_4'/>
-        <origin xyz='${-wheel_steer_to_wheel_length/2+wheel_steer_length/2} 0 ${-wheel_steer_to_wheel_height/2-wheel_steer_height/2}' rpy='0 0 0'/>
+        <origin xyz='${wheel_steer_to_wheel_length/2-wheel_steer_length/2} 0 ${-wheel_steer_to_wheel_height/2-wheel_steer_height/2}' rpy='0 0 0'/>
     </joint>
 </robot>

Commit message: Wheels

File: ros2_ws/src/my_rover/urdf/wheel.xacro (robot description, xacro)
@@ -231,4 +231,7 @@
                 <box size='${wheel_steer_to_wheel_length} ${wheel_steer_to_wheel_width} ${wheel_steer_to_wheel_height}'/>
             </geometry>
+            <material name='gray'>
+                <color rgba='0.5 0.5 0.5 1.0'/>
+            </material>
         </visual>
         <collision>
@@ -250,4 +253,7 @@
                 <box size='${wheel_steer_to_wheel_length} ${wheel_steer_to_wheel_width} ${wheel_steer_to_wheel_height}'/>
             </geometry>
+            <material name='gray'>
+                <color rgba='0.5 0.5 0.5 1.0'/>
+            </material>
         </visual>
         <collision>
@@ -269,4 +275,7 @@
                 <box size='${wheel_steer_to_wheel_length} ${wheel_steer_to_wheel_width} ${wheel_steer_to_wheel_height}'/>
             </geometry>
+            <material name='gray'>
+                <color rgba='0.5 0.5 0.5 1.0'/>
+            </material>
         </visual>
         <collision>
@@ -288,4 +297,7 @@
                 <box size='${wheel_steer_to_wheel_length} ${wheel_steer_to_wheel_width} ${wheel_steer_to_wheel_height}'/>
             </geometry>
+            <material name='gray'>
+                <color rgba='0.5 0.5 0.5 1.0'/>
+            </material>
         </visual>
         <collision>
@@ -321,3 +333,115 @@
         <origin xyz='${wheel_steer_to_wheel_length/2-wheel_steer_length/2} 0 ${-wheel_steer_to_wheel_height/2-wheel_steer_height/2}' rpy='0 0 0'/>
     </joint>
+    <link name='wheel'>
+        <visual>
+            <geometry>
+                <origin xyz='0 0 0' rpy='0 0 0'/>
+                <cylinder radius='${wheel_base_radius}' length='${wheel_base_length}'/>
+            </geometry>
+            <material name='gray'>
+                <color rgba='0.5 0.5 0.5 1.0'/>
+            </material>
+        </visual>
+        <collision>
+            <origin xyz='0 0 0' rpy='0 0 0'/>
+            <geometry>
+                <cylinder radius='${wheel_base_radius}' length='${wheel_base_length}'/>
+            </geometry>
+        </collision>
+        <inertial>
+            <origin xyz='0 0 0' rpy='0 0 0'/>
+            <mass value='1'/>
+            <xacro:cylinder_inertia m="1" r="${wheel_base_radius}" h="${wheel_base_length}"/>
+        </inertial>
+    </link>
+    <link name='wheel_2'>
+        <visual>
+            <geometry>
+                <origin xyz='0 0 0' rpy='0 0 0'/>
+                <cylinder radius='${wheel_base_radius}' length='${wheel_base_length}'/>
+            </geometry>
+            <material name='gray'>
+                <color rgba='0.5 0.5 0.5 1.0'/>
+            </material>
+        </visual>
+        <collision>
+            <origin xyz='0 0 0' rpy='0 0 0'/>
+            <geometry>
+                <cylinder radius='${wheel_base_radius}' length='${wheel_base_length}'/>
+            </geometry>
+        </collision>
+        <inertial>
+            <origin xyz='0 0 0' rpy='0 0 0'/>
+            <mass value='1'/>
+            <xacro:cylinder_inertia m="1" r="${wheel_base_radius}" h="${wheel_base_length}"/>
+        </inertial>
+    </link>
+    <link name='wheel_3'>
+        <visual>
+            <geometry>
+                <origin xyz='0 0 0' rpy='0 0 0'/>
+                <cylinder radius='${wheel_base_radius}' length='${wheel_base_length}'/>
+            </geometry>
+            <material name='gray'>
+                <color rgba='0.5 0.5 0.5 1.0'/>
+            </material>
+        </visual>
+        <collision>
+            <origin xyz='0 0 0' rpy='0 0 0'/>
+            <geometry>
+                <cylinder radius='${wheel_base_radius}' length='${wheel_base_length}'/>
+            </geometry>
+        </collision>
+        <inertial>
+            <origin xyz='0 0 0' rpy='0 0 0'/>
+            <mass value='1'/>
+            <xacro:cylinder_inertia m="1" r="${wheel_base_radius}" h="${wheel_base_length}"/>
+        </inertial>
+    </link>
+    <link name='wheel_4'>
+        <visual>
+            <geometry>
+                <origin xyz='0 0 0' rpy='0 0 0'/>
+                <cylinder radius='${wheel_base_radius}' length='${wheel_base_length}'/>
+            </geometry>
+            <material name='gray'>
+                <color rgba='0.5 0.5 0.5 1.0'/>
+            </material>
+        </visual>
+        <collision>
+            <origin xyz='0 0 0' rpy='0 0 0'/>
+            <geometry>
+                <cylinder radius='${wheel_base_radius}' length='${wheel_base_length}'/>
+            </geometry>
+        </collision>
+        <inertial>
+            <origin xyz='0 0 0' rpy='0 0 0'/>
+            <mass value='1'/>
+            <xacro:cylinder_inertia m="1" r="${wheel_base_radius}" h="${wheel_base_length}"/>
+        </inertial>
+    </link>
+    <joint name='wheel_joint' type='continous'>
+        <parent link='wheel_steer_to_wheel'/>
+        <child link='wheel'/>
+        <origin xyz='0.2 0.4 0.8' rpy='0 1.5707 0'/>
+        <axis xyz='1 0 0'/>
+    </joint>
+    <joint name='wheel_joint_2' type='continous'>
+        <parent link='wheel_steer_to_wheel_2'/>
+        <child link='wheel_2'/>
+        <origin xyz='0 0 0' rpy='0 1.5707 0'/>
+        <axis xyz='1 0 0'/>
+    </joint>
+    <joint name='wheel_joint_3' type='continous'>
+        <parent link='wheel_steer_to_wheel_3'/>
+        <child link='wheel_3'/>
+        <origin xyz='0 0 0' rpy='0 1.5707 0'/>
+        <axis xyz='1 0 0'/>
+    </joint>
+    <joint name='wheel_joint_4' type='continous'>
+        <parent link='wheel_steer_to_wheel_4'/>
+        <child link='wheel_4'/>
+        <origin xyz='0 0 0' rpy='0 1.5707 0'/>
+        <axis xyz='1 0 0'/>
+    </joint>
 </robot>

Commit message: Wheels

File: ros2_ws/src/my_rover/urdf/wheel.xacro (robot description, xacro)
@@ -335,6 +335,6 @@
     <link name='wheel'>
         <visual>
-            <geometry>
-                <origin xyz='0 0 0' rpy='0 0 0'/>
+            <origin xyz='0 0 0' rpy='0 0 0'/>
+            <geometry>
                 <cylinder radius='${wheel_base_radius}' length='${wheel_base_length}'/>
             </geometry>
@@ -357,6 +357,6 @@
     <link name='wheel_2'>
         <visual>
-            <geometry>
-                <origin xyz='0 0 0' rpy='0 0 0'/>
+            <origin xyz='0 0 0' rpy='0 0 0'/>
+            <geometry>
                 <cylinder radius='${wheel_base_radius}' length='${wheel_base_length}'/>
             </geometry>
@@ -379,6 +379,6 @@
     <link name='wheel_3'>
         <visual>
-            <geometry>
-                <origin xyz='0 0 0' rpy='0 0 0'/>
+            <origin xyz='0 0 0' rpy='0 0 0'/>
+            <geometry>
                 <cylinder radius='${wheel_base_radius}' length='${wheel_base_length}'/>
             </geometry>
@@ -401,25 +401,25 @@
     <link name='wheel_4'>
         <visual>
-            <geometry>
-                <origin xyz='0 0 0' rpy='0 0 0'/>
-                <cylinder radius='${wheel_base_radius}' length='${wheel_base_length}'/>
-            </geometry>
-            <material name='gray'>
-                <color rgba='0.5 0.5 0.5 1.0'/>
-            </material>
-        </visual>
-        <collision>
-            <origin xyz='0 0 0' rpy='0 0 0'/>
-            <geometry>
-                <cylinder radius='${wheel_base_radius}' length='${wheel_base_length}'/>
-            </geometry>
-        </collision>
-        <inertial>
-            <origin xyz='0 0 0' rpy='0 0 0'/>
-            <mass value='1'/>
-            <xacro:cylinder_inertia m="1" r="${wheel_base_radius}" h="${wheel_base_length}"/>
-        </inertial>
-    </link>
-    <joint name='wheel_joint' type='continous'>
+            <origin xyz='0 0 0' rpy='0 0 0'/>
+            <geometry>
+                <cylinder radius='${wheel_base_radius}' length='${wheel_base_length}'/>
+            </geometry>
+            <material name='gray'>
+                <color rgba='0.5 0.5 0.5 1.0'/>
+            </material>
+        </visual>
+        <collision>
+            <origin xyz='0 0 0' rpy='0 0 0'/>
+            <geometry>
+                <cylinder radius='${wheel_base_radius}' length='${wheel_base_length}'/>
+            </geometry>
+        </collision>
+        <inertial>
+            <origin xyz='0 0 0' rpy='0 0 0'/>
+            <mass value='1'/>
+            <xacro:cylinder_inertia m="1" r="${wheel_base_radius}" h="${wheel_base_length}"/>
+        </inertial>
+    </link>
+    <joint name='wheel_joint' type='continuous'>
         <parent link='wheel_steer_to_wheel'/>
         <child link='wheel'/>
@@ -427,5 +427,5 @@
         <axis xyz='1 0 0'/>
     </joint>
-    <joint name='wheel_joint_2' type='continous'>
+    <joint name='wheel_joint_2' type='continuous'>
         <parent link='wheel_steer_to_wheel_2'/>
         <child link='wheel_2'/>
@@ -433,5 +433,5 @@
         <axis xyz='1 0 0'/>
     </joint>
-    <joint name='wheel_joint_3' type='continous'>
+    <joint name='wheel_joint_3' type='continuous'>
         <parent link='wheel_steer_to_wheel_3'/>
         <child link='wheel_3'/>
@@ -439,5 +439,5 @@
         <axis xyz='1 0 0'/>
     </joint>
-    <joint name='wheel_joint_4' type='continous'>
+    <joint name='wheel_joint_4' type='continuous'>
         <parent link='wheel_steer_to_wheel_4'/>
         <child link='wheel_4'/>

Commit message: Wheels

File: ros2_ws/src/my_rover/urdf/wheel.xacro (robot description, xacro)
@@ -430,5 +430,5 @@
         <parent link='wheel_steer_to_wheel_2'/>
         <child link='wheel_2'/>
-        <origin xyz='0 0 0' rpy='0 1.5707 0'/>
+        <origin xyz='${wheel_steer_to_wheel_length/2+wheel_length/2} 0 ${-wheel_steer_to_wheel_height/2}' rpy='0 1.5707 0'/>
         <axis xyz='0 0 1'/>
     </joint>
@@ -436,5 +436,5 @@
         <parent link='wheel_steer_to_wheel_3'/>
         <child link='wheel_3'/>
-        <origin xyz='0 0 0' rpy='0 1.5707 0'/>
+        <origin xyz='${wheel_steer_to_wheel_length/2+wheel_length/2} 0 ${-wheel_steer_to_wheel_height/2}' rpy='0 1.5707 0'/>
         <axis xyz='0 0 1'/>
     </joint>
@@ -442,5 +442,5 @@
         <parent link='wheel_steer_to_wheel_4'/>
         <child link='wheel_4'/>
-        <origin xyz='0 0 0' rpy='0 1.5707 0'/>
+        <origin xyz='${wheel_steer_to_wheel_length/2+wheel_length/2} 0 ${-wheel_steer_to_wheel_height/2}' rpy='0 1.5707 0'/>
         <axis xyz='0 0 1'/>
     </joint>

Commit message: Wheels

File: ros2_ws/src/my_rover/urdf/wheel.xacro (robot description, xacro)
@@ -430,5 +430,5 @@
         <parent link='wheel_steer_to_wheel_2'/>
         <child link='wheel_2'/>
-        <origin xyz='${wheel_steer_to_wheel_length/2+wheel_length/2} 0 ${-wheel_steer_to_wheel_height/2}' rpy='0 1.5707 0'/>
+        <origin xyz='${-wheel_steer_to_wheel_length/2-wheel_length/2} 0 ${-wheel_steer_to_wheel_height/2}' rpy='0 1.5707 0'/>
         <axis xyz='0 0 1'/>
     </joint>
@@ -436,5 +436,5 @@
         <parent link='wheel_steer_to_wheel_3'/>
         <child link='wheel_3'/>
-        <origin xyz='${wheel_steer_to_wheel_length/2+wheel_length/2} 0 ${-wheel_steer_to_wheel_height/2}' rpy='0 1.5707 0'/>
+        <origin xyz='${-wheel_steer_to_wheel_length/2-wheel_length/2} 0 ${-wheel_steer_to_wheel_height/2}' rpy='0 1.5707 0'/>
         <axis xyz='0 0 1'/>
     </joint>
