Commit message: Suspension_rods

File: ros2_ws/src/my_rover/urdf/suspension.xacro (robot description, xacro)
@@ -43,5 +43,5 @@
         <child link='chassis_suspension_rod'/>
         <origin xyz='0 ${chassis_width/2+ chassis_suspension_rod_length} 0' rpy='${pi/2} 0 0'/>
-        <axis xyz='0 0 0'/>
+        <axis xyz='0 0 1'/>
         <limit lower='-1.57' upper='1.57' effort='1000' velocity='1'/>
     </joint>
@@ -50,5 +50,5 @@
         <child link='chassis_suspension_rod_2'/>
         <origin xyz='0 ${-chassis_width/2 - chassis_suspension_rod_length} 0' rpy='${pi/2} 0 0'/>
-        <axis xyz='0 0 0'/>
+        <axis xyz='0 0 1'/>
         <limit lower='-1.57' upper='1.57' effort='1000' velocity='1'/>
     </joint>

Commit message: Suspension_rods

File: ros2_ws/src/my_rover/urdf/suspension.xacro (robot description, xacro)
@@ -5,5 +5,5 @@
             <origin xyz='0 0 0' rpy='0 0 0'/>
             <geometry>
-                <cylinder radius='${chassis_suspension_rod_radius}' height='${chassis_suspension_rod_length}'/>
+                <cylinder radius='${chassis_suspension_rod_radius}' length='${chassis_suspension_rod_length}'/>
             </geometry>
         </visual>
@@ -11,5 +11,5 @@
             <origin xyz='0 0 0' rpy='0 0 0'/>
             <geometry>
-                <cylinder radius='${chassis_suspension_rod_radius}' height='${chassis_suspension_rod_length}'/>
+                <cylinder radius='${chassis_suspension_rod_radius}' length='${chassis_suspension_rod_length}'/>
             </geometry>
         </collision>
@@ -24,5 +24,5 @@
             <origin xyz='0 0 0' rpy='0 0 0'/>
             <geometry>
-                <cylinder radius='${chassis_suspension_rod_radius}' height='${chassis_suspension_rod_length}'/>
+                <cylinder radius='${chassis_suspension_rod_radius}' length='${chassis_suspension_rod_length}'/>
             </geometry>
         </visual>
@@ -30,5 +30,5 @@
             <origin xyz='0 0 0' rpy='0 0 0'/>
             <geometry>
-                <cylinder radius='${chassis_suspension_rod_radius}' height='${chassis_suspension_rod_length}'/>
+                <cylinder radius='${chassis_suspension_rod_radius}' length='${chassis_suspension_rod_length}'/>
             </geometry>
         </collision>

Commit message: Suspension_rod

File: ros2_ws/src/my_rover/urdf/suspension.xacro (robot description, xacro)
@@ -55,5 +55,5 @@
     <link name='suspension_rod'>
         <visual>
-            <origin xyz='0 0 {-chassis_suspension_rod_length/2}' rpy='0 0 0'/>
+            <origin xyz='0 0 ${-chassis_suspension_rod_length/2}' rpy='0 0 0'/>
             <geometry>
                 <cylinder radius='${suspension_rod_radius}' length='${suspension_rod_length}'/>

Commit message: Suspension_rod

File: ros2_ws/src/my_rover/urdf/suspension.xacro (robot description, xacro)
@@ -55,5 +55,5 @@
     <link name='suspension_rod'>
         <visual>
-            <origin xyz='0 0 ${-chassis_suspension_rod_length/2}' rpy='0 0 0'/>
+            <origin xyz='0 0 ${-suspension_rod_length/2}' rpy='0 0 0'/>
             <geometry>
                 <cylinder radius='${suspension_rod_radius}' length='${suspension_rod_length}'/>

Commit message: Suspension_rod

File: ros2_ws/src/my_rover/urdf/suspension.xacro (robot description, xacro)
@@ -55,5 +55,5 @@
     <link name='suspension_rod'>
         <visual>
-            <origin xyz='0 0 ${-suspension_rod_length/2}' rpy='0 0 0'/>
+            <origin xyz='0 0 ${suspension_rod_length/2}' rpy='0 0 0'/>
             <geometry>
                 <cylinder radius='${suspension_rod_radius}' length='${suspension_rod_length}'/>
@@ -132,5 +132,5 @@
         <parent link='chassis_suspension_rod'/>
         <child link='suspension_rod'/>
-        <origin xyz='0 0 0' rpy='0 ${2*pi/3} 0'/>
+        <origin xyz='0 0 0' rpy='${pi/3} ${pi/2} 0'/>
     </joint>
     <joint name='suspension_rod_2_joint' type='fixed'>

Commit message: Suspension_rods

File: ros2_ws/src/my_rover/urdf/suspension.xacro (robot description, xacro)
@@ -132,5 +132,5 @@
         <parent link='chassis_suspension_rod'/>
         <child link='suspension_rod'/>
-        <origin xyz='0 0 0' rpy='${-pi/6} ${pi/2} 0'/>
+        <origin xyz='0 0 0' rpy='${pi/6} ${-pi/2} 0'/>
     </joint>
     <joint name='suspension_rod_2_joint' type='fixed'>

Commit message: Suspension_rod

File: ros2_ws/src/my_rover/urdf/suspension.xacro (robot description, xacro)
@@ -132,5 +132,5 @@
         <parent link='chassis_suspension_rod'/>
         <child link='suspension_rod'/>
-        <origin xyz='0 0 0' rpy='${pi/3} ${pi/2} 0'/>
+        <origin xyz='0 0 0' rpy='${-pi/6} ${pi/2} 0'/>
     </joint>
     <joint name='suspension_rod_2_joint' type='fixed'>

Commit message: Suspension_rod

File: ros2_ws/src/my_rover/urdf/suspension.xacro (robot description, xacro)
@@ -74,5 +74,5 @@
     <link name='suspension_rod_2'>
         <visual>
-            <origin xyz='0 0 0' rpy='0 0 0'/>
+            <origin xyz='0 0 ${suspension_rod_length/2}' rpy='0 0 0'/>
             <geometry>
                 <cylinder radius='${suspension_rod_radius}' length='${suspension_rod_length}'/>
@@ -93,5 +93,5 @@
     <link name='suspension_rod_3'>
         <visual>
-            <origin xyz='0 0 0' rpy='0 0 0'/>
+            <origin xyz='0 0 ${suspension_rod_length/2}' rpy='0 0 0'/>
             <geometry>
                 <cylinder radius='${suspension_rod_radius}' length='${suspension_rod_length}'/>
@@ -112,5 +112,5 @@
     <link name='suspension_rod_4'>
         <visual>
-            <origin xyz='0 0 0' rpy='0 0 0'/>
+            <origin xyz='0 0 ${suspension_rod_length/2}' rpy='0 0 0'/>
             <geometry>
                 <cylinder radius='${suspension_rod_radius}' length='${suspension_rod_length}'/>
@@ -137,15 +137,15 @@
         <parent link='chassis_suspension_rod_2'/>
         <child link='suspension_rod_2'/>
-        <origin xyz='0 0 0' rpy='0 ${2*pi/3} 0'/>
+        <origin xyz='0 0 0' rpy='${atan2(chassis_height/2 ,chassis_length/2)} ${-pi/2} 0'/>
     </joint>
     <joint name='suspension_rod_3_joint' type='fixed'>
         <parent link='chassis_suspension_rod'/>
         <child link='suspension_rod_3'/>
-        <origin xyz='0 0 0' rpy='0 ${4*pi/3} 0'/>
+        <origin xyz='0 0 0' rpy='${atan2(chassis_height/2 ,chassis_length/2)} ${pi/2} 0'/>
     </joint>
     <joint name='suspension_rod_4_joint' type='fixed'>
         <parent link='chassis_suspension_rod_2'/>
         <child link='suspension_rod_4'/>
-        <origin xyz='0 0 0' rpy='0 ${4*pi/3} 0'/>
+        <origin xyz='0 0 0' rpy='${atan2(chassis_height/2 ,chassis_length/2)} ${pi/2} 0'/>
     </joint>
 </robot>

Commit message: Suspension_rod

File: ros2_ws/src/my_rover/urdf/suspension.xacro (robot description, xacro)
@@ -142,5 +142,5 @@
         <parent link='chassis_suspension_rod'/>
         <child link='suspension_rod_3'/>
-        <origin xyz='${chassis_suspension_rod_length/3} 0 0' rpy='${atan2(chassis_height/2 ,chassis_length/2)} ${pi/2} 0'/>
+        <origin xyz='0 ${chassis_suspension_rod_length/3} 0' rpy='${atan2(chassis_height/2 ,chassis_length/2)} ${pi/2} 0'/>
     </joint>
     <joint name='suspension_rod_4_joint' type='fixed'>

Commit message: Suspension_rod

File: ros2_ws/src/my_rover/urdf/suspension.xacro (robot description, xacro)
@@ -142,5 +142,5 @@
         <parent link='chassis_suspension_rod'/>
         <child link='suspension_rod_3'/>
-        <origin xyz='0 ${chassis_suspension_rod_length/3} 0' rpy='${atan2(chassis_height/2 ,chassis_length/2)} ${pi/2} 0'/>
+        <origin xyz='0 0 ${chassis_suspension_rod_length/3}' rpy='${atan2(chassis_height/2 ,chassis_length/2)} ${pi/2} 0'/>
     </joint>
     <joint name='suspension_rod_4_joint' type='fixed'>

Commit message: Suspension_rod

File: ros2_ws/src/my_rover/urdf/suspension.xacro (robot description, xacro)
@@ -132,20 +132,20 @@
         <parent link='chassis_suspension_rod'/>
         <child link='suspension_rod'/>
-        <origin xyz='0 0 0' rpy='${atan2(chassis_height/2 ,chassis_length/2)} ${-pi/2} 0'/>
+        <origin xyz='0 0 ${-chassis_suspension_rod_length/3}' rpy='${atan2(chassis_height/2 ,chassis_length/2)} ${-pi/2} 0'/>
     </joint>
     <joint name='suspension_rod_2_joint' type='fixed'>
         <parent link='chassis_suspension_rod_2'/>
         <child link='suspension_rod_2'/>
-        <origin xyz='0 0 0' rpy='${atan2(chassis_height/2 ,chassis_length/2)} ${-pi/2} 0'/>
+        <origin xyz='0 0 ${-chassis_suspension_rod_length/3}' rpy='${atan2(chassis_height/2 ,chassis_length/2)} ${-pi/2} 0'/>
     </joint>
     <joint name='suspension_rod_3_joint' type='fixed'>
         <parent link='chassis_suspension_rod'/>
         <child link='suspension_rod_3'/>
-        <origin xyz='0 0 ${chassis_suspension_rod_length/3}' rpy='${atan2(chassis_height/2 ,chassis_length/2)} ${pi/2} 0'/>
+        <origin xyz='0 0 ${-chassis_suspension_rod_length/3}' rpy='${atan2(chassis_height/2 ,chassis_length/2)} ${pi/2} 0'/>
     </joint>
     <joint name='suspension_rod_4_joint' type='fixed'>
         <parent link='chassis_suspension_rod_2'/>
         <child link='suspension_rod_4'/>
-        <origin xyz='0 0 0' rpy='${atan2(chassis_height/2 ,chassis_length/2)} ${pi/2} 0'/>
+        <origin xyz='0 0 ${-chassis_suspension_rod_length/3}' rpy='${atan2(chassis_height/2 ,chassis_length/2)} ${pi/2} 0'/>
     </joint>
 </robot>

Commit message: Suspension_rod

File: ros2_ws/src/my_rover/urdf/suspension.xacro (robot description, xacro)
@@ -142,10 +142,10 @@
         <parent link='chassis_suspension_rod'/>
         <child link='suspension_rod_3'/>
-        <origin xyz='0 0 ${-chassis_suspension_rod_length/3}' rpy='${atan2(chassis_height/2 ,chassis_length/2)} ${pi/2} 0'/>
+        <origin xyz='0 0 ${chassis_suspension_rod_length/3}' rpy='${atan2(chassis_height/2 ,chassis_length/2)} ${pi/2} 0'/>
     </joint>
     <joint name='suspension_rod_4_joint' type='fixed'>
         <parent link='chassis_suspension_rod_2'/>
         <child link='suspension_rod_4'/>
-        <origin xyz='0 0 ${-chassis_suspension_rod_length/3}' rpy='${atan2(chassis_height/2 ,chassis_length/2)} ${pi/2} 0'/>
+        <origin xyz='0 0 ${chassis_suspension_rod_length/3}' rpy='${atan2(chassis_height/2 ,chassis_length/2)} ${pi/2} 0'/>
     </joint>
 </robot>

Commit message: Suspension_rod

File: ros2_ws/src/my_rover/urdf/suspension.xacro (robot description, xacro)
@@ -137,10 +137,10 @@
         <parent link='chassis_suspension_rod_2'/>
         <child link='suspension_rod_2'/>
-        <origin xyz='0 0 ${-chassis_suspension_rod_length/3}' rpy='${atan2(chassis_height/2 ,chassis_length/2)} ${-pi/2} 0'/>
+        <origin xyz='0 0 ${chassis_suspension_rod_length/3}' rpy='${atan2(chassis_height/2 ,chassis_length/2)} ${-pi/2} 0'/>
     </joint>
     <joint name='suspension_rod_3_joint' type='fixed'>
         <parent link='chassis_suspension_rod'/>
         <child link='suspension_rod_3'/>
-        <origin xyz='0 0 ${chassis_suspension_rod_length/3}' rpy='${atan2(chassis_height/2 ,chassis_length/2)} ${pi/2} 0'/>
+        <origin xyz='0 0 ${-chassis_suspension_rod_length/3}' rpy='${atan2(chassis_height/2 ,chassis_length/2)} ${pi/2} 0'/>
     </joint>
     <joint name='suspension_rod_4_joint' type='fixed'>

Commit message: Wheels

File: ros2_ws/src/my_rover/urdf/suspension.xacro (robot description, xacro)
@@ -61,5 +61,5 @@
         </visual>
         <collision>
-            <origin xyz='0 0 0' rpy='0 0 0'/>
+            <origin xyz='0 0 ${suspension_rod_length/2}' rpy='0 0 0'/>
             <geometry>
                 <cylinder radius='${suspension_rod_radius}' length='${suspension_rod_length}'/>
@@ -67,5 +67,5 @@
         </collision>
         <inertial>
-            <origin xyz='0 0 0' rpy='0 0 0'/>
+            <origin xyz='0 0 ${suspension_rod_length/2}' rpy='0 0 0'/>
             <mass value='1'/>
             <xacro:cylinder_inertia m='1' r='${suspension_rod_radius}' h='${suspension_rod_length}'/>
@@ -80,5 +80,5 @@
         </visual>
         <collision>
-            <origin xyz='0 0 0' rpy='0 0 0'/>
+            <origin xyz='0 0 ${suspension_rod_length/2}' rpy='0 0 0'/>
             <geometry>
                 <cylinder radius='${suspension_rod_radius}' length='${suspension_rod_length}'/>
@@ -86,5 +86,5 @@
         </collision>
         <inertial>
-            <origin xyz='0 0 0' rpy='0 0 0'/>
+            <origin xyz='0 0 ${suspension_rod_length/2}' rpy='0 0 0'/>
             <mass value='1'/>
             <xacro:cylinder_inertia m='1' r='${suspension_rod_radius}' h='${suspension_rod_length}'/>
@@ -99,5 +99,5 @@
         </visual>
         <collision>
-            <origin xyz='0 0 0' rpy='0 0 0'/>
+            <origin xyz='0 0 ${suspension_rod_length/2}' rpy='0 0 0'/>
             <geometry>
                 <cylinder radius='${suspension_rod_radius}' length='${suspension_rod_length}'/>
@@ -105,5 +105,5 @@
         </collision>
         <inertial>
-            <origin xyz='0 0 0' rpy='0 0 0'/>
+            <origin xyz='0 0 ${suspension_rod_length/2}' rpy='0 0 0'/>
             <mass value='1'/>
             <xacro:cylinder_inertia m='1' r='${suspension_rod_radius}' h='${suspension_rod_length}'/>
@@ -118,5 +118,5 @@
         </visual>
         <collision>
-            <origin xyz='0 0 0' rpy='0 0 0'/>
+            <origin xyz='0 0 ${suspension_rod_length/2}' rpy='0 0 0'/>
             <geometry>
                 <cylinder radius='${suspension_rod_radius}' length='${suspension_rod_length}'/>
@@ -124,5 +124,5 @@
         </collision>
         <inertial>
-            <origin xyz='0 0 0' rpy='0 0 0'/>
+            <origin xyz='0 0 ${suspension_rod_length/2}' rpy='0 0 0'/>
             <mass value='1'/>
             <xacro:cylinder_inertia m='1' r='${suspension_rod_radius}' h='${suspension_rod_length}'/>

File: ros2_ws/src/my_rover/urdf/wheel.xacro (robot description, xacro)
@@ -3,109 +3,109 @@
     <link name='wheel-base'>
         <visual>
-            <origin xyz='0 0 0' rpy='0 0 0'/>
+            <origin xyz='0 0 ${wheel_base_length/2}' rpy='0 0 0'/>
             <geometry>
                 <cylinder radius='${wheel_base_radius}' length='${wheel_base_length}'/>
-                <material name='black'>
-                    <color rgba='0.2 0.2 0.2 1.0'/>
-                </material>
             </geometry>
-            <collision>
-                <origin xyz='0 0 0' rpy='0 0 0'/>
-                <geometry>
-                    <cylinder radius='${wheel_base_radius}' length='${wheel_base_length}'/>
-                </geometry>
-            </collision>
-            <inertial>
-                <origin xyz='0 0 0' rpy='0 0 0'/>
-                <mass value='1'/>
-                <xacro:cylinder_inertia m="1" r="${wheel_base_radius}" h="${wheel_base_length}"/>
-            </inertial>
+            <material name='black'>
+                <color rgba='0.2 0.2 0.2 1.0'/>
+            </material>
         </visual>
+        <collision>
+            <origin xyz='0 0 ${wheel_base_length/2}' rpy='0 0 0'/>
+            <geometry>
+                <cylinder radius='${wheel_base_radius}' length='${wheel_base_length}'/>
+            </geometry>
+        </collision>
+        <inertial>
+            <origin xyz='0 0 ${wheel_base_length/2}' rpy='0 0 0'/>
+            <mass value='1'/>
+            <xacro:cylinder_inertia m="1" r="${wheel_base_radius}" h="${wheel_base_length}"/>
+        </inertial>
     </link>
     <link name='wheel-base_2'>
         <visual>
-            <origin xyz='0 0 0' rpy='0 0 0'/>
+            <origin xyz='0 0 ${wheel_base_length/2}' rpy='0 0 0'/>
             <geometry>
                 <cylinder radius='${wheel_base_radius}' length='${wheel_base_length}'/>
-                <material name='black'>
-                    <color rgba='0.2 0.2 0.2 1.0'/>
-                </material>
             </geometry>
-            <collision>
-                <origin xyz='0 0 0' rpy='0 0 0'/>
-                <geometry>
-                    <cylinder radius='${wheel_base_radius}' length='${wheel_base_length}'/>
-                </geometry>
-            </collision>
-            <inertial>
-                <origin xyz='0 0 0' rpy='0 0 0'/>
-                <mass value='1'/>
-                <xacro:cylinder_inertia m="1" r="${wheel_base_radius}" h="${wheel_base_length}"/>
-            </inertial>
+            <material name='black'>
+                <color rgba='0.2 0.2 0.2 1.0'/>
+            </material>
         </visual>
+        <collision>
+            <origin xyz='0 0 ${wheel_base_length/2}' rpy='0 0 0'/>
+            <geometry>
+                <cylinder radius='${wheel_base_radius}' length='${wheel_base_length}'/>
+            </geometry>
+        </collision>
+        <inertial>
+            <origin xyz='0 0 ${wheel_base_length/2}' rpy='0 0 0'/>
+            <mass value='1'/>
+            <xacro:cylinder_inertia m="1" r="${wheel_base_radius}" h="${wheel_base_length}"/>
+        </inertial>
     </link>
     <link name='wheel-base_3'>
         <visual>
-            <origin xyz='0 0 0' rpy='0 0 0'/>
+            <origin xyz='0 0 ${wheel_base_length/2}' rpy='0 0 0'/>
             <geometry>
                 <cylinder radius='${wheel_base_radius}' length='${wheel_base_length}'/>
-                <material name='black'>
-                    <color rgba='0.2 0.2 0.2 1.0'/>
-                </material>
             </geometry>
-            <collision>
-                <origin xyz='0 0 0' rpy='0 0 0'/>
-                <geometry>
-                    <cylinder radius='${wheel_base_radius}' length='${wheel_base_length}'/>
-                </geometry>
-            </collision>
-            <inertial>
-                <origin xyz='0 0 0' rpy='0 0 0'/>
-                <mass value='1'/>
-                <xacro:cylinder_inertia m="1" r="${wheel_base_radius}" h="${wheel_base_length}"/>
-            </inertial>
+            <material name='black'>
+                <color rgba='0.2 0.2 0.2 1.0'/>
+            </material>
         </visual>
+        <collision>
+            <origin xyz='0 0 ${wheel_base_length/2}' rpy='0 0 0'/>
+            <geometry>
+                <cylinder radius='${wheel_base_radius}' length='${wheel_base_length}'/>
+            </geometry>
+        </collision>
+        <inertial>
+            <origin xyz='0 0 ${wheel_base_length/2}' rpy='0 0 0'/>
+            <mass value='1'/>
+            <xacro:cylinder_inertia m="1" r="${wheel_base_radius}" h="${wheel_base_length}"/>
+        </inertial>
     </link>
     <link name='wheel-base_4'>
         <visual>
-            <origin xyz='0 0 0' rpy='0 0 0'/>
+            <origin xyz='0 0 ${wheel_base_length/2}' rpy='0 0 0'/>
             <geometry>
                 <cylinder radius='${wheel_base_radius}' length='${wheel_base_length}'/>
-                <material name='black'>
-                    <color rgba='0.2 0.2 0.2 1.0'/>
-                </material>
             </geometry>
-            <collision>
-                <origin xyz='0 0 0' rpy='0 0 0'/>
-                <geometry>
-                    <cylinder radius='${wheel_base_radius}' length='${wheel_base_length}'/>
-                </geometry>
-            </collision>
-            <inertial>
-                <origin xyz='0 0 0' rpy='0 0 0'/>
-                <mass value='1'/>
-                <xacro:cylinder_inertia m="1" r="${wheel_base_radius}" h="${wheel_base_length}"/>
-            </inertial>
+            <material name='black'>
+                <color rgba='0.2 0.2 0.2 1.0'/>
+            </material>
         </visual>
+        <collision>
+            <origin xyz='0 0 ${wheel_base_length/2}' rpy='0 0 0'/>
+            <geometry>
+                <cylinder radius='${wheel_base_radius}' length='${wheel_base_length}'/>
+            </geometry>
+        </collision>
+        <inertial>
+            <origin xyz='0 0 ${wheel_base_length/2}' rpy='0 0 0'/>
+            <mass value='1'/>
+            <xacro:cylinder_inertia m="1" r="${wheel_base_radius}" h="${wheel_base_length}"/>
+        </inertial>
     </link>
     <joint name='wheel_base_joint' type='fixed'>
         <parent link='suspension_rod'/>
         <child link='wheel-base'/>
-        <origin xyz='0 0 ${suspension_rod_length}' rpy='${pi/2 - atan2(chassis_height/2 ,chassis_length/2)} 0 0'/>
+        <origin xyz='0 0 ${suspension_rod_length}' rpy='${-pi/2 - atan2(chassis_height/2 ,chassis_length/2)} 0 0'/>
     </joint>
     <joint name='wheel_base_2_joint' type='fixed'>
         <parent link='suspension_rod_2'/>
         <child link='wheel-base_2'/>
-        <origin xyz='0 0 ${suspension_rod_length}' rpy='0 0 0'/>
+        <origin xyz='0 0 ${suspension_rod_length}' rpy='${-pi/2 - atan2(chassis_height/2 ,chassis_length/2)} 0 0'/>
     </joint>
     <joint name='wheel_base_3_joint' type='fixed'>
         <parent link='suspension_rod_3'/>
         <child link='wheel-base_3'/>
-        <origin xyz='0 0 ${suspension_rod_length}' rpy='0 0 0'/>
+        <origin xyz='0 0 ${suspension_rod_length}' rpy='${-pi/2 - atan2(chassis_height/2 ,chassis_length/2)} 0 0'/>
     </joint>
     <joint name='wheel_base_4_joint' type='fixed'>
         <parent link='suspension_rod_4'/>
         <child link='wheel-base_4'/>
-        <origin xyz='0 0 ${suspension_rod_length}' rpy='0 0 0'/>
+        <origin xyz='0 0 ${suspension_rod_length}' rpy='${-pi/2 - atan2(chassis_height/2 ,chassis_length/2)} 0 0'/>
     </joint>
 </robot>
