Commit message: Wheels

File: ros2_ws/src/my_rover/urdf/suspension.xacro (robot description, xacro)
@@ -150,20 +150,20 @@
         <parent link='chassis_suspension_rod'/>
         <child link='suspension_rod'/>
-        <origin xyz='0 0 ${-chassis_suspension_rod_length/3}' rpy='${atan2((chassis_height/2-wheel_base_lenght) ,(chassis_length/2-wheel_base_radius))} ${-pi/2} 0'/>
+        <origin xyz='0 0 ${-chassis_suspension_rod_length/3}' rpy='${atan2((chassis_height/2-wheel_base_length) ,(chassis_length/2-wheel_base_radius))} ${-pi/2} 0'/>
     </joint>
     <joint name='suspension_rod_2_joint' type='fixed'>
         <parent link='chassis_suspension_rod_2'/>
         <child link='suspension_rod_2'/>
-        <origin xyz='0 0 ${chassis_suspension_rod_length/3}' rpy='${atan2((chassis_height/2-wheel_base_lenght) ,(chassis_length/2-wheel_base_radius))} ${-pi/2} 0'/>
+        <origin xyz='0 0 ${chassis_suspension_rod_length/3}' rpy='${atan2((chassis_height/2-wheel_base_length) ,(chassis_length/2-wheel_base_radius))} ${-pi/2} 0'/>
     </joint>
     <joint name='suspension_rod_3_joint' type='fixed'>
         <parent link='chassis_suspension_rod'/>
         <child link='suspension_rod_3'/>
-        <origin xyz='0 0 ${-chassis_suspension_rod_length/3}' rpy='${atan2((chassis_height/2-wheel_base_lenght) ,(chassis_length/2-wheel_base_radius))} ${pi/2} 0'/>
+        <origin xyz='0 0 ${-chassis_suspension_rod_length/3}' rpy='${atan2((chassis_height/2-wheel_base_length) ,(chassis_length/2-wheel_base_radius))} ${pi/2} 0'/>
     </joint>
     <joint name='suspension_rod_4_joint' type='fixed'>
         <parent link='chassis_suspension_rod_2'/>
         <child link='suspension_rod_4'/>
-        <origin xyz='0 0 ${chassis_suspension_rod_length/3}' rpy='${atan2((chassis_height/2-wheel_base_lenght) ,(chassis_length/2-wheel_base_radius))} ${pi/2} 0'/>
+        <origin xyz='0 0 ${chassis_suspension_rod_length/3}' rpy='${atan2((chassis_height/2-wheel_base_length) ,(chassis_length/2-wheel_base_radius))} ${pi/2} 0'/>
     </joint>
 </robot>
