Commit message: Chassis

File: ros2_ws/src/my_rover/urdf/rover_properties.xacro (robot description, xacro)
@@ -1,6 +1,6 @@
 <?xml version="1.0"?>
 <robot xmlns:xacro='http://www.ros.org/wiki/xacro' name='my_rover'>
-    <xacro:property name='chassis_length' value='1.5'/>
+    <xacro:property name='chassis_length' value='1.25'/>
     <xacro:property name='chassis_width' value='1'/>
-    <xacro:property name='chassis_height' value='1'/>
+    <xacro:property name='chassis_height' value='0.5'/>
 </robot>

Commit message: Suspension_rods

File: ros2_ws/src/my_rover/urdf/rover_properties.xacro (robot description, xacro)
@@ -4,5 +4,7 @@
     <xacro:property name='chassis_width' value='1'/>
     <xacro:property name='chassis_height' value='0.5'/>
-    <xacro:property name='chassis_suspension_rod_length' value='0.1'/>
-    <xacro:property name='chassis_suspension_rod_radius' value='0.05'/>
+    <xacro:property name='chassis_suspension_rod_length' value='0.5'/>
+    <xacro:property name='chassis_suspension_rod_radius' value='0.02'/>
+    <xacro:property name='suspension_rod_length' value='1'/>
+    <xacro:property name='suspension_rod_radius' value='0.02'/>
 </robot>

File: ros2_ws/src/my_rover/urdf/suspension.xacro (robot description, xacro)
@@ -42,5 +42,5 @@
         <parent link='chassis'/>
         <child link='chassis_suspension_rod'/>
-        <origin xyz='0 ${chassis_width/2+ chassis_suspension_rod_length} 0' rpy='${pi/2} 0 0'/>
+        <origin xyz='0 ${chassis_width/2+ chassis_suspension_rod_length/2} 0' rpy='${pi/2} 0 0'/>
         <axis xyz='0 0 1'/>
         <limit lower='-1.57' upper='1.57' effort='1000' velocity='1'/>
@@ -49,7 +49,103 @@
         <parent link='chassis'/>
         <child link='chassis_suspension_rod_2'/>
-        <origin xyz='0 ${-chassis_width/2 - chassis_suspension_rod_length} 0' rpy='${pi/2} 0 0'/>
+        <origin xyz='0 ${-chassis_width/2 - chassis_suspension_rod_length/2} 0' rpy='${pi/2} 0 0'/>
         <axis xyz='0 0 1'/>
         <limit lower='-1.57' upper='1.57' effort='1000' velocity='1'/>
     </joint>
+    <link name='suspension_rod'>
+        <visual>
+            <origin xyz='0 0 0' rpy='0 0 0'/>
+            <geometry>
+                <cylinder radius='${suspension_rod_radius}' length='${suspension_rod_length}'/>
+            </geometry>
+        </visual>
+        <collision>
+            <origin xyz='0 0 0' rpy='0 0 0'/>
+            <geometry>
+                <cylinder radius='${suspension_rod_radius}' length='${suspension_rod_length}'/>
+            </geometry>
+        </collision>
+        <inertial>
+            <origin xyz='0 0 0' rpy='0 0 0'/>
+            <mass value='1'/>
+            <xacro:cylinder_inertia m='1' r='${suspension_rod_radius}' h='${suspension_rod_length}'/>
+        </inertial>
+    </link>
+    <link name='suspension_rod_2'>
+        <visual>
+            <origin xyz='0 0 0' rpy='0 0 0'/>
+            <geometry>
+                <cylinder radius='${suspension_rod_radius}' length='${suspension_rod_length}'/>
+            </geometry>
+        </visual>
+        <collision>
+            <origin xyz='0 0 0' rpy='0 0 0'/>
+            <geometry>
+                <cylinder radius='${suspension_rod_radius}' length='${suspension_rod_length}'/>
+            </geometry>
+        </collision>
+        <inertial>
+            <origin xyz='0 0 0' rpy='0 0 0'/>
+            <mass value='1'/>
+            <xacro:cylinder_inertia m='1' r='${suspension_rod_radius}' h='${suspension_rod_length}'/>
+        </inertial>
+    </link>
+    <link name='suspension_rod_3'>
+        <visual>
+            <origin xyz='0 0 0' rpy='0 0 0'/>
+            <geometry>
+                <cylinder radius='${suspension_rod_radius}' length='${suspension_rod_length}'/>
+            </geometry>
+        </visual>
+        <collision>
+            <origin xyz='0 0 0' rpy='0 0 0'/>
+            <geometry>
+                <cylinder radius='${suspension_rod_radius}' length='${suspension_rod_length}'/>
+            </geometry>
+        </collision>
+        <inertial>
+            <origin xyz='0 0 0' rpy='0 0 0'/>
+            <mass value='1'/>
+            <xacro:cylinder_inertia m='1' r='${suspension_rod_radius}' h='${suspension_rod_length}'/>
+        </inertial>
+    </link>
+    <link name='suspension_rod_4'>
+        <visual>
+            <origin xyz='0 0 0' rpy='0 0 0'/>
+            <geometry>
+                <cylinder radius='${suspension_rod_radius}' length='${suspension_rod_length}'/>
+            </geometry>
+        </visual>
+        <collision>
+            <origin xyz='0 0 0' rpy='0 0 0'/>
+            <geometry>
+                <cylinder radius='${suspension_rod_radius}' length='${suspension_rod_length}'/>
+            </geometry>
+        </collision>
+        <inertial>
+            <origin xyz='0 0 0' rpy='0 0 0'/>
+            <mass value='1'/>
+            <xacro:cylinder_inertia m='1' r='${suspension_rod_radius}' h='${suspension_rod_length}'/>
+        </inertial>
+    </link>
+    <joint name='suspension_rod_joint' type='fixed'>
+        <parent link='chassis_suspension_rod'/>
+        <child link='suspension_rod'/>
+        <origin xyz='0 0 0' rpy='0 ${2*pi/3} 0'/>
+    </joint>
+    <joint name='suspension_rod_2_joint' type='fixed'>
+        <parent link='chassis_suspension_rod_2'/>
+        <child link='suspension_rod_2'/>
+        <origin xyz='0 0 0' rpy='0 ${2*pi/3} 0'/>
+    </joint>
+    <joint name='suspension_rod_3_joint' type='fixed'>
+        <parent link='chassis_suspension_rod'/>
+        <child link='suspension_rod_3'/>
+        <origin xyz='0 0 0' rpy='0 ${4*pi/3} 0'/>
+    </joint>
+    <joint name='suspension_rod_4_joint' type='fixed'>
+        <parent link='chassis_suspension_rod_2'/>
+        <child link='suspension_rod_4'/>
+        <origin xyz='0 0 0' rpy='0 ${4*pi/3} 0'/>
+    </joint>
 </robot>

Commit message: Suspension_rods

File: ros2_ws/src/my_rover/urdf/rover_properties.xacro (robot description, xacro)
@@ -4,5 +4,5 @@
     <xacro:property name='chassis_width' value='1'/>
     <xacro:property name='chassis_height' value='0.5'/>
-    <xacro:property name='chassis_suspension_rod_length' value='0.5'/>
+    <xacro:property name='chassis_suspension_rod_length' value='0.05'/>
     <xacro:property name='chassis_suspension_rod_radius' value='0.02'/>
     <xacro:property name='suspension_rod_length' value='1'/>

File: ros2_ws/src/my_rover/urdf/suspension.xacro (robot description, xacro)
@@ -55,5 +55,5 @@
     <link name='suspension_rod'>
         <visual>
-            <origin xyz='0 0 0' rpy='0 0 0'/>
+            <origin xyz='0 0 {-chassis_suspension_rod_length/2}' rpy='0 0 0'/>
             <geometry>
                 <cylinder radius='${suspension_rod_radius}' length='${suspension_rod_length}'/>

Commit message: Suspension_rod

File: ros2_ws/src/my_rover/urdf/rover_properties.xacro (robot description, xacro)
@@ -6,5 +6,5 @@
     <xacro:property name='chassis_suspension_rod_length' value='0.05'/>
     <xacro:property name='chassis_suspension_rod_radius' value='0.02'/>
-    <xacro:property name='suspension_rod_length' value='1'/>
+    <xacro:property name='suspension_rod_length' value='${sqrt((chassis_length/2)**2 + (chassis_height/2)**2)}'/>
     <xacro:property name='suspension_rod_radius' value='0.02'/>
 </robot>

File: ros2_ws/src/my_rover/urdf/suspension.xacro (robot description, xacro)
@@ -132,5 +132,5 @@
         <parent link='chassis_suspension_rod'/>
         <child link='suspension_rod'/>
-        <origin xyz='0 0 0' rpy='${pi/6} ${-pi/2} 0'/>
+        <origin xyz='0 0 0' rpy='${atan2(chassis_height/2 ,chassis_length/2)} ${-pi/2} 0'/>
     </joint>
     <joint name='suspension_rod_2_joint' type='fixed'>

Commit message: Suspension_rod

File: ros2_ws/src/my_rover/urdf/rover_properties.xacro (robot description, xacro)
@@ -4,5 +4,5 @@
     <xacro:property name='chassis_width' value='1'/>
     <xacro:property name='chassis_height' value='0.5'/>
-    <xacro:property name='chassis_suspension_rod_length' value='0.05'/>
+    <xacro:property name='chassis_suspension_rod_length' value='0.1'/>
     <xacro:property name='chassis_suspension_rod_radius' value='0.02'/>
     <xacro:property name='suspension_rod_length' value='${sqrt((chassis_length/2)**2 + (chassis_height/2)**2)}'/>

File: ros2_ws/src/my_rover/urdf/suspension.xacro (robot description, xacro)
@@ -142,5 +142,5 @@
         <parent link='chassis_suspension_rod'/>
         <child link='suspension_rod_3'/>
-        <origin xyz='0 0 0' rpy='${atan2(chassis_height/2 ,chassis_length/2)} ${pi/2} 0'/>
+        <origin xyz='${chassis_suspension_rod_length/3} 0 0' rpy='${atan2(chassis_height/2 ,chassis_length/2)} ${pi/2} 0'/>
     </joint>
     <joint name='suspension_rod_4_joint' type='fixed'>

Commit message: Wheels

File: ros2_ws/src/my_rover/urdf/rover_properties.xacro (robot description, xacro)
@@ -8,3 +8,5 @@
     <xacro:property name='suspension_rod_length' value='${sqrt((chassis_length/2)**2 + (chassis_height/2)**2)}'/>
     <xacro:property name='suspension_rod_radius' value='0.02'/>
+    <xacro:property name='wheel_base_lenght' value='0.08'/>
+    <xacro:property name='wheel_base_radius' value='0.05'/>
 </robot>

Commit message: Wheels

File: ros2_ws/src/my_rover/urdf/rover_properties.xacro (robot description, xacro)
@@ -8,5 +8,5 @@
     <xacro:property name='suspension_rod_length' value='${sqrt((chassis_length/2)**2 + (chassis_height/2)**2)}'/>
     <xacro:property name='suspension_rod_radius' value='0.02'/>
-    <xacro:property name='wheel_base_lenght' value='0.08'/>
+    <xacro:property name='wheel_base_length' value='0.08'/>
     <xacro:property name='wheel_base_radius' value='0.05'/>
 </robot>

Commit message: Wheels

File: ros2_ws/src/my_rover/urdf/rover_properties.xacro (robot description, xacro)
@@ -8,5 +8,5 @@
     <xacro:property name='suspension_rod_length' value='${sqrt((chassis_length/2)**2 + (chassis_height/2)**2)}'/>
     <xacro:property name='suspension_rod_radius' value='0.02'/>
-    <xacro:property name='wheel_base_length' value='0.08'/>
-    <xacro:property name='wheel_base_radius' value='0.05'/>
+    <xacro:property name='wheel_base_length' value='0.065'/>
+    <xacro:property name='wheel_base_radius' value='0.065'/>
 </robot>

File: ros2_ws/src/my_rover/urdf/suspension.xacro (robot description, xacro)
@@ -7,4 +7,7 @@
                 <cylinder radius='${chassis_suspension_rod_radius}' length='${chassis_suspension_rod_length}'/>
             </geometry>
+            <material name='gray'>
+                <color rgba='0.5 0.5 0.5 1.0'/>
+            </material>
         </visual>
         <collision>
@@ -26,4 +29,7 @@
                 <cylinder radius='${chassis_suspension_rod_radius}' length='${chassis_suspension_rod_length}'/>
             </geometry>
+            <material name='gray'>
+                <color rgba='0.5 0.5 0.5 1.0'/>
+            </material>
         </visual>
         <collision>
@@ -59,4 +65,7 @@
                 <cylinder radius='${suspension_rod_radius}' length='${suspension_rod_length}'/>
             </geometry>
+            <material name='gray'>
+                <color rgba='0.5 0.5 0.5 1.0'/>
+            </material>
         </visual>
         <collision>
@@ -78,4 +87,7 @@
                 <cylinder radius='${suspension_rod_radius}' length='${suspension_rod_length}'/>
             </geometry>
+            <material name='gray'>
+                <color rgba='0.5 0.5 0.5 1.0'/>
+            </material>
         </visual>
         <collision>
@@ -97,4 +109,7 @@
                 <cylinder radius='${suspension_rod_radius}' length='${suspension_rod_length}'/>
             </geometry>
+            <material name='gray'>
+                <color rgba='0.5 0.5 0.5 1.0'/>
+            </material>
         </visual>
         <collision>
@@ -116,4 +131,7 @@
                 <cylinder radius='${suspension_rod_radius}' length='${suspension_rod_length}'/>
             </geometry>
+            <material name='gray'>
+                <color rgba='0.5 0.5 0.5 1.0'/>
+            </material>
         </visual>
         <collision>

File: ros2_ws/src/my_rover/urdf/wheel.xacro (robot description, xacro)
@@ -7,6 +7,6 @@
                 <cylinder radius='${wheel_base_radius}' length='${wheel_base_length}'/>
             </geometry>
-            <material name='black'>
-                <color rgba='0.2 0.2 0.2 1.0'/>
+            <material name='gray'>
+                <color rgba='0.5 0.5 0.5 1.0'/>
             </material>
         </visual>
@@ -29,6 +29,6 @@
                 <cylinder radius='${wheel_base_radius}' length='${wheel_base_length}'/>
             </geometry>
-            <material name='black'>
-                <color rgba='0.2 0.2 0.2 1.0'/>
+            <material name='gray'>
+                <color rgba='0.5 0.5 0.5 1.0'/>
             </material>
         </visual>
@@ -51,6 +51,6 @@
                 <cylinder radius='${wheel_base_radius}' length='${wheel_base_length}'/>
             </geometry>
-            <material name='black'>
-                <color rgba='0.2 0.2 0.2 1.0'/>
+            <material name='gray'>
+                <color rgba='0.5 0.5 0.5 1.0'/>
             </material>
         </visual>
@@ -73,6 +73,6 @@
                 <cylinder radius='${wheel_base_radius}' length='${wheel_base_length}'/>
             </geometry>
-            <material name='black'>
-                <color rgba='0.2 0.2 0.2 1.0'/>
+            <material name='gray'>
+                <color rgba='0.5 0.5 0.5 1.0'/>
             </material>
         </visual>

Commit message: Wheels

File: ros2_ws/src/my_rover/urdf/rover_properties.xacro (robot description, xacro)
@@ -10,3 +10,6 @@
     <xacro:property name='wheel_base_length' value='0.065'/>
     <xacro:property name='wheel_base_radius' value='0.065'/>
+    <xacro:property name='wheel_steer_length' value='0.03'/>
+    <xacro:property name='wheel_steer_width' value='0.05'/>
+    <xacro:property name='wheel_steer_height' value='0.08'/>
 </robot>

Commit message: Wheels

File: ros2_ws/src/my_rover/urdf/rover_properties.xacro (robot description, xacro)
@@ -10,6 +10,6 @@
     <xacro:property name='wheel_base_length' value='0.065'/>
     <xacro:property name='wheel_base_radius' value='0.065'/>
-    <xacro:property name='wheel_steer_length' value='0.03'/>
-    <xacro:property name='wheel_steer_width' value='0.05'/>
-    <xacro:property name='wheel_steer_height' value='0.08'/>
+    <xacro:property name='wheel_steer_length' value='0.06'/>
+    <xacro:property name='wheel_steer_width' value='0.07'/>
+    <xacro:property name='wheel_steer_height' value='0.03'/>
 </robot>

Commit message: Wheels

File: ros2_ws/src/my_rover/urdf/rover_properties.xacro (robot description, xacro)
@@ -12,4 +12,7 @@
     <xacro:property name='wheel_steer_length' value='0.06'/>
     <xacro:property name='wheel_steer_width' value='0.07'/>
-    <xacro:property name='wheel_steer_height' value='0.03'/>
+    <xacro:property name='wheel_steer_height' value='0.02'/>
+    <xacro:property name='wheel_steer_to_wheel_length' value='0.1'/>
+    <xacro:property name='wheel_steer_to_wheel_width' value='0.05'/>
+    <xacro:property name='wheel_steer_to_wheel_height' value='0.07'/>
 </robot>

File: ros2_ws/src/my_rover/urdf/wheel.xacro (robot description, xacro)
@@ -207,5 +207,5 @@
         <parent link='wheel-base_2'/>
         <child link='wheel_steer_2'/>
-        <origin xyz='0 0 ${-wheel_base_length/3}' rpy='0 0 0'/>
+        <origin xyz='0 0 ${-2*wheel_base_length/3 - wheel_steer_height/2}' rpy='0 0 0'/>
         <axis xyz='0 0 1'/>
         <limit lower='-1.57' upper='1.57' effort='1000' velocity='1'/>
@@ -214,5 +214,5 @@
         <parent link='wheel-base_3'/>
         <child link='wheel_steer_3'/>
-        <origin xyz='0 0 ${-wheel_base_length/3}' rpy='0 0 0'/>
+        <origin xyz='0 0 ${-2*wheel_base_length/3 - wheel_steer_height/2}' rpy='0 0 0'/>
         <axis xyz='0 0 1'/>
         <limit lower='-1.57' upper='1.57' effort='1000' velocity='1'/>
@@ -221,7 +221,103 @@
         <parent link='wheel-base_4'/>
         <child link='wheel_steer_4'/>
-        <origin xyz='0 0 ${-wheel_base_length/3}' rpy='0 0 0'/>
+        <origin xyz='0 0 ${-2*wheel_base_length/3 - wheel_steer_height/2}' rpy='0 0 0'/>
         <axis xyz='0 0 1'/>
         <limit lower='-1.57' upper='1.57' effort='1000' velocity='1'/>
     </joint>
+    <link name='wheel_steer_to_wheel'>
+        <visual>
+            <origin xyz='0 0 0' rpy='0 0 0'/>
+            <geometry>
+                <box size='${wheel_steer_to_wheel_length} ${wheel_steer_to_width} ${wheel_steer_to_height}'/>
+            </geometry>
+        </visual>
+        <collision>
+            <origin xyz='0 0 0' rpy='0 0 0'/>
+            <geometry>
+                <box size='${wheel_steer_to_wheel_length} ${wheel_steer_to_width} ${wheel_steer_to_height}'/>
+            </geometry>
+        </collision>
+        <inertial>
+            <origin xyz='0 0 0' rpy='0 0 0'/>
+            <mass value='1'/>
+            <xacro:box_inertia m="1" x="${wheel_steer_to_wheel_length}" y="${wheel_steer_to_width}" z="${wheel_steer_to_height}"/>
+        </inertial>
+    </link>
+    <link name='wheel_steer_to_wheel_2'>
+        <visual>
+            <origin xyz='0 0 0' rpy='0 0 0'/>
+            <geometry>
+                <box size='${wheel_steer_to_wheel_length} ${wheel_steer_to_width} ${wheel_steer_to_height}'/>
+            </geometry>
+        </visual>
+        <collision>
+            <origin xyz='0 0 0' rpy='0 0 0'/>
+            <geometry>
+                <box size='${wheel_steer_to_wheel_length} ${wheel_steer_to_width} ${wheel_steer_to_height}'/>
+            </geometry>
+        </collision>
+        <inertial>
+            <origin xyz='0 0 0' rpy='0 0 0'/>
+            <mass value='1'/>
+            <xacro:box_inertia m="1" x="${wheel_steer_to_wheel_length}" y="${wheel_steer_to_width}" z="${wheel_steer_to_height}"/>
+        </inertial>
+    </link>
+    <link name='wheel_steer_to_wheel_3'>
+        <visual>
+            <origin xyz='0 0 0' rpy='0 0 0'/>
+            <geometry>
+                <box size='${wheel_steer_to_wheel_length} ${wheel_steer_to_width} ${wheel_steer_to_height}'/>
+            </geometry>
+        </visual>
+        <collision>
+            <origin xyz='0 0 0' rpy='0 0 0'/>
+            <geometry>
+                <box size='${wheel_steer_to_wheel_length} ${wheel_steer_to_width} ${wheel_steer_to_height}'/>
+            </geometry>
+        </collision>
+        <inertial>
+            <origin xyz='0 0 0' rpy='0 0 0'/>
+            <mass value='1'/>
+            <xacro:box_inertia m="1" x="${wheel_steer_to_wheel_length}" y="${wheel_steer_to_width}" z="${wheel_steer_to_height}"/>
+        </inertial>
+    </link>
+    <link name='wheel_steer_to_wheel_4'>
+        <visual>
+            <origin xyz='0 0 0' rpy='0 0 0'/>
+            <geometry>
+                <box size='${wheel_steer_to_wheel_length} ${wheel_steer_to_width} ${wheel_steer_to_height}'/>
+            </geometry>
+        </visual>
+        <collision>
+            <origin xyz='0 0 0' rpy='0 0 0'/>
+            <geometry>
+                <box size='${wheel_steer_to_wheel_length} ${wheel_steer_to_width} ${wheel_steer_to_height}'/>
+            </geometry>
+        </collision>
+        <inertial>
+            <origin xyz='0 0 0' rpy='0 0 0'/>
+            <mass value='1'/>
+            <xacro:box_inertia m="1" x="${wheel_steer_to_wheel_length}" y="${wheel_steer_to_width}" z="${wheel_steer_to_height}"/>
+        </inertial>
+    </link>
+    <joint name='wheel_steer_to_wheel_joint_1' type='fixed'>
+        <parent link='wheel_steer'/>
+        <child link='wheel_steer_to_wheel'/>
+        <origin xyz='0.5 0.35 1' rpy='0 0 0'/>
+    </joint>
+    <joint name='wheel_steer_to_wheel_joint_2' type='fixed'>
+        <parent link='wheel_steer_2'/>
+        <child link='wheel_steer_to_wheel_2'/>
+        <origin xyz='0 0 0' rpy='0 0 0'/>
+    </joint>
+    <joint name='wheel_steer_to_wheel_joint_3' type='fixed'>
+        <parent link='wheel_steer_3'/>
+        <child link='wheel_steer_to_wheel_3'/>
+        <origin xyz='0 0 0' rpy='0 0 0'/>
+    </joint>
+    <joint name='wheel_steer_to_wheel_joint_4' type='fixed'>
+        <parent link='wheel_steer_4'/>
+        <child link='wheel_steer_to_wheel_4'/>
+        <origin xyz='0 0 0' rpy='0 0 0'/>
+    </joint>
 </robot>

Commit message: Wheels

File: ros2_ws/src/my_rover/urdf/rover_properties.xacro (robot description, xacro)
@@ -13,6 +13,6 @@
     <xacro:property name='wheel_steer_width' value='0.07'/>
     <xacro:property name='wheel_steer_height' value='0.02'/>
-    <xacro:property name='wheel_steer_to_wheel_length' value='0.1'/>
-    <xacro:property name='wheel_steer_to_wheel_width' value='0.05'/>
-    <xacro:property name='wheel_steer_to_wheel_height' value='0.07'/>
+    <xacro:property name='wheel_steer_to_wheel_length' value='0.05'/>
+    <xacro:property name='wheel_steer_to_wheel_width' value='0.1'/>
+    <xacro:property name='wheel_steer_to_wheel_height' value='0.5'/>
 </robot>

File: ros2_ws/src/my_rover/urdf/wheel.xacro (robot description, xacro)
@@ -221,5 +221,5 @@
         <parent link='wheel-base_4'/>
         <child link='wheel_steer_4'/>
-        <origin xyz='0 0 ${-2*wheel_base_length/3 - wheel_steer_height/2}' rpy='0 0 0'/>
+        <origin xyz='0 0 ${-2*wheel_base_length/3 - wheel_steer_height}' rpy='0 0 0'/>
         <axis xyz='0 0 1'/>
         <limit lower='-1.57' upper='1.57' effort='1000' velocity='1'/>
