Commit message: Wheels

File: ros2_ws/src/my_rover/urdf/rover_properties.xacro (robot description, xacro)
@@ -10,8 +10,8 @@
     <xacro:property name='wheel_base_length' value='0.065'/>
     <xacro:property name='wheel_base_radius' value='0.065'/>
-    <xacro:property name='wheel_steer_length' value='0.06'/>
+    <xacro:property name='wheel_steer_length' value='0.1'/>
     <xacro:property name='wheel_steer_width' value='0.07'/>
     <xacro:property name='wheel_steer_height' value='0.02'/>
-    <xacro:property name='wheel_steer_to_wheel_length' value='0.05'/>
+    <xacro:property name='wheel_steer_to_wheel_length' value='0.04'/>
     <xacro:property name='wheel_steer_to_wheel_width' value='0.1'/>
     <xacro:property name='wheel_steer_to_wheel_height' value='0.5'/>

File: ros2_ws/src/my_rover/urdf/wheel.xacro (robot description, xacro)
@@ -200,5 +200,5 @@
         <parent link='wheel-base'/>
         <child link='wheel_steer'/>
-        <origin xyz='0 0 ${-2*wheel_base_length/3 - wheel_steer_height/2}' rpy='0 0 0'/>
+        <origin xyz='0 0 ${-2*wheel_base_length/3 - wheel_steer_height}' rpy='0 0 0'/>
         <axis xyz='0 0 1'/>
         <limit lower='-1.57' upper='1.57' effort='1000' velocity='1'/>
@@ -207,5 +207,5 @@
         <parent link='wheel-base_2'/>
         <child link='wheel_steer_2'/>
-        <origin xyz='0 0 ${-2*wheel_base_length/3 - wheel_steer_height/2}' rpy='0 0 0'/>
+        <origin xyz='0 0 ${-2*wheel_base_length/3 - wheel_steer_height}' rpy='0 0 0'/>
         <axis xyz='0 0 1'/>
         <limit lower='-1.57' upper='1.57' effort='1000' velocity='1'/>
@@ -214,5 +214,5 @@
         <parent link='wheel-base_3'/>
         <child link='wheel_steer_3'/>
-        <origin xyz='0 0 ${-2*wheel_base_length/3 - wheel_steer_height/2}' rpy='0 0 0'/>
+        <origin xyz='0 0 ${-2*wheel_base_length/3 - wheel_steer_height}' rpy='0 0 0'/>
         <axis xyz='0 0 1'/>
         <limit lower='-1.57' upper='1.57' effort='1000' velocity='1'/>
@@ -304,5 +304,5 @@
         <parent link='wheel_steer'/>
         <child link='wheel_steer_to_wheel'/>
-        <origin xyz='0.5 0.35 1' rpy='0 0 0'/>
+        <origin xyz='${wheel_steer_to_wheel_length/2-wheel_steer_length/2} 0 ${-wheel_steer_to_wheel_height/2-wheel_steer_height/2}' rpy='0 0 0'/>
     </joint>
     <joint name='wheel_steer_to_wheel_joint_2' type='fixed'>

Commit message: Wheels

File: ros2_ws/src/my_rover/urdf/rover_properties.xacro (robot description, xacro)
@@ -14,5 +14,5 @@
     <xacro:property name='wheel_steer_height' value='0.02'/>
     <xacro:property name='wheel_steer_to_wheel_length' value='0.04'/>
-    <xacro:property name='wheel_steer_to_wheel_width' value='0.1'/>
-    <xacro:property name='wheel_steer_to_wheel_height' value='0.5'/>
+    <xacro:property name='wheel_steer_to_wheel_width' value='0.07'/>
+    <xacro:property name='wheel_steer_to_wheel_height' value='0.1'/>
 </robot>

Commit message: Wheels

File: ros2_ws/src/my_rover/urdf/rover_properties.xacro (robot description, xacro)
@@ -10,5 +10,5 @@
     <xacro:property name='wheel_base_length' value='0.065'/>
     <xacro:property name='wheel_base_radius' value='0.065'/>
-    <xacro:property name='wheel_steer_length' value='0.1'/>
+    <xacro:property name='wheel_steer_length' value='0.085'/>
     <xacro:property name='wheel_steer_width' value='0.07'/>
     <xacro:property name='wheel_steer_height' value='0.02'/>

Commit message: Wheels

File: ros2_ws/src/my_rover/urdf/rover_properties.xacro (robot description, xacro)
@@ -15,4 +15,4 @@
     <xacro:property name='wheel_steer_to_wheel_length' value='0.04'/>
     <xacro:property name='wheel_steer_to_wheel_width' value='0.07'/>
-    <xacro:property name='wheel_steer_to_wheel_height' value='0.1'/>
+    <xacro:property name='wheel_steer_to_wheel_height' value='0.15'/>
 </robot>

File: ros2_ws/src/my_rover/urdf/wheel.xacro (robot description, xacro)
@@ -309,15 +309,15 @@
         <parent link='wheel_steer_2'/>
         <child link='wheel_steer_to_wheel_2'/>
-        <origin xyz='0 0 0' rpy='0 0 0'/>
+        <origin xyz='${wheel_steer_to_wheel_length/2-wheel_steer_length/2} 0 ${-wheel_steer_to_wheel_height/2-wheel_steer_height/2}' rpy='0 0 0'/>
     </joint>
     <joint name='wheel_steer_to_wheel_joint_3' type='fixed'>
         <parent link='wheel_steer_3'/>
         <child link='wheel_steer_to_wheel_3'/>
-        <origin xyz='0 0 0' rpy='0 0 0'/>
+        <origin xyz='${wheel_steer_to_wheel_length/2-wheel_steer_length/2} 0 ${-wheel_steer_to_wheel_height/2-wheel_steer_height/2}' rpy='0 0 0'/>
     </joint>
     <joint name='wheel_steer_to_wheel_joint_4' type='fixed'>
         <parent link='wheel_steer_4'/>
         <child link='wheel_steer_to_wheel_4'/>
-        <origin xyz='0 0 0' rpy='0 0 0'/>
+        <origin xyz='${wheel_steer_to_wheel_length/2-wheel_steer_length/2} 0 ${-wheel_steer_to_wheel_height/2-wheel_steer_height/2}' rpy='0 0 0'/>
     </joint>
 </robot>

Commit message: Wheels

File: ros2_ws/src/my_rover/urdf/rover_properties.xacro (robot description, xacro)
@@ -16,3 +16,5 @@
     <xacro:property name='wheel_steer_to_wheel_width' value='0.07'/>
     <xacro:property name='wheel_steer_to_wheel_height' value='0.15'/>
+    <xacro:property name='wheel_lenght' value='0.65'/>
+    <xacro:property name='wheel_radius' value='${wheel_steer_to_wheel_height*0.9}'/>
 </robot>

File: ros2_ws/src/my_rover/urdf/wheel.xacro (robot description, xacro)
@@ -424,6 +424,6 @@
         <parent link='wheel_steer_to_wheel'/>
         <child link='wheel'/>
-        <origin xyz='0.2 0.4 0.8' rpy='0 1.5707 0'/>
-        <axis xyz='1 0 0'/>
+        <origin xyz='${wheel_steer_to_wheel_length/2+wheel_lenght/2} 0 ${-wheel_steer_to_wheel_height/2}' rpy='0 1.5707 0'/>
+        <axis xyz='0 0 1'/>
     </joint>
     <joint name='wheel_joint_2' type='continuous'>
@@ -431,5 +431,5 @@
         <child link='wheel_2'/>
         <origin xyz='0 0 0' rpy='0 1.5707 0'/>
-        <axis xyz='1 0 0'/>
+        <axis xyz='0 0 1'/>
     </joint>
     <joint name='wheel_joint_3' type='continuous'>
@@ -437,5 +437,5 @@
         <child link='wheel_3'/>
         <origin xyz='0 0 0' rpy='0 1.5707 0'/>
-        <axis xyz='1 0 0'/>
+        <axis xyz='0 0 1'/>
     </joint>
     <joint name='wheel_joint_4' type='continuous'>
@@ -443,5 +443,5 @@
         <child link='wheel_4'/>
         <origin xyz='0 0 0' rpy='0 1.5707 0'/>
-        <axis xyz='1 0 0'/>
+        <axis xyz='0 0 1'/>
     </joint>
 </robot>

Commit message: Wheels

File: ros2_ws/src/my_rover/urdf/rover_properties.xacro (robot description, xacro)
@@ -16,5 +16,5 @@
     <xacro:property name='wheel_steer_to_wheel_width' value='0.07'/>
     <xacro:property name='wheel_steer_to_wheel_height' value='0.15'/>
-    <xacro:property name='wheel_lenght' value='0.65'/>
+    <xacro:property name='wheel_length' value='0.065'/>
     <xacro:property name='wheel_radius' value='${wheel_steer_to_wheel_height*0.9}'/>
 </robot>

File: ros2_ws/src/my_rover/urdf/wheel.xacro (robot description, xacro)
@@ -337,20 +337,20 @@
             <origin xyz='0 0 0' rpy='0 0 0'/>
             <geometry>
-                <cylinder radius='${wheel_base_radius}' length='${wheel_base_length}'/>
-            </geometry>
-            <material name='gray'>
-                <color rgba='0.5 0.5 0.5 1.0'/>
-            </material>
-        </visual>
-        <collision>
-            <origin xyz='0 0 0' rpy='0 0 0'/>
-            <geometry>
-                <cylinder radius='${wheel_base_radius}' length='${wheel_base_length}'/>
-            </geometry>
-        </collision>
-        <inertial>
-            <origin xyz='0 0 0' rpy='0 0 0'/>
-            <mass value='1'/>
-            <xacro:cylinder_inertia m="1" r="${wheel_base_radius}" h="${wheel_base_length}"/>
+                <cylinder radius='${wheel_radius}' length='${wheel_base_length}'/>
+            </geometry>
+            <material name='gray'>
+                <color rgba='0.5 0.5 0.5 1.0'/>
+            </material>
+        </visual>
+        <collision>
+            <origin xyz='0 0 0' rpy='0 0 0'/>
+            <geometry>
+                <cylinder radius='${wheel_radius}' length='${wheel_base_length}'/>
+            </geometry>
+        </collision>
+        <inertial>
+            <origin xyz='0 0 0' rpy='0 0 0'/>
+            <mass value='1'/>
+            <xacro:cylinder_inertia m="1" r="${wheel_radius}" h="${wheel_base_length}"/>
         </inertial>
     </link>
@@ -359,20 +359,20 @@
             <origin xyz='0 0 0' rpy='0 0 0'/>
             <geometry>
-                <cylinder radius='${wheel_base_radius}' length='${wheel_base_length}'/>
-            </geometry>
-            <material name='gray'>
-                <color rgba='0.5 0.5 0.5 1.0'/>
-            </material>
-        </visual>
-        <collision>
-            <origin xyz='0 0 0' rpy='0 0 0'/>
-            <geometry>
-                <cylinder radius='${wheel_base_radius}' length='${wheel_base_length}'/>
-            </geometry>
-        </collision>
-        <inertial>
-            <origin xyz='0 0 0' rpy='0 0 0'/>
-            <mass value='1'/>
-            <xacro:cylinder_inertia m="1" r="${wheel_base_radius}" h="${wheel_base_length}"/>
+                <cylinder radius='${wheel_radius}' length='${wheel_base_length}'/>
+            </geometry>
+            <material name='gray'>
+                <color rgba='0.5 0.5 0.5 1.0'/>
+            </material>
+        </visual>
+        <collision>
+            <origin xyz='0 0 0' rpy='0 0 0'/>
+            <geometry>
+                <cylinder radius='${wheel_radius}' length='${wheel_base_length}'/>
+            </geometry>
+        </collision>
+        <inertial>
+            <origin xyz='0 0 0' rpy='0 0 0'/>
+            <mass value='1'/>
+            <xacro:cylinder_inertia m="1" r="${wheel_radius}" h="${wheel_base_length}"/>
         </inertial>
     </link>
@@ -381,20 +381,20 @@
             <origin xyz='0 0 0' rpy='0 0 0'/>
             <geometry>
-                <cylinder radius='${wheel_base_radius}' length='${wheel_base_length}'/>
-            </geometry>
-            <material name='gray'>
-                <color rgba='0.5 0.5 0.5 1.0'/>
-            </material>
-        </visual>
-        <collision>
-            <origin xyz='0 0 0' rpy='0 0 0'/>
-            <geometry>
-                <cylinder radius='${wheel_base_radius}' length='${wheel_base_length}'/>
-            </geometry>
-        </collision>
-        <inertial>
-            <origin xyz='0 0 0' rpy='0 0 0'/>
-            <mass value='1'/>
-            <xacro:cylinder_inertia m="1" r="${wheel_base_radius}" h="${wheel_base_length}"/>
+                <cylinder radius='${wheel_radius}' length='${wheel_base_length}'/>
+            </geometry>
+            <material name='gray'>
+                <color rgba='0.5 0.5 0.5 1.0'/>
+            </material>
+        </visual>
+        <collision>
+            <origin xyz='0 0 0' rpy='0 0 0'/>
+            <geometry>
+                <cylinder radius='${wheel_radius}' length='${wheel_base_length}'/>
+            </geometry>
+        </collision>
+        <inertial>
+            <origin xyz='0 0 0' rpy='0 0 0'/>
+            <mass value='1'/>
+            <xacro:cylinder_inertia m="1" r="${wheel_radius}" h="${wheel_base_length}"/>
         </inertial>
     </link>
@@ -403,20 +403,20 @@
             <origin xyz='0 0 0' rpy='0 0 0'/>
             <geometry>
-                <cylinder radius='${wheel_base_radius}' length='${wheel_base_length}'/>
-            </geometry>
-            <material name='gray'>
-                <color rgba='0.5 0.5 0.5 1.0'/>
-            </material>
-        </visual>
-        <collision>
-            <origin xyz='0 0 0' rpy='0 0 0'/>
-            <geometry>
-                <cylinder radius='${wheel_base_radius}' length='${wheel_base_length}'/>
-            </geometry>
-        </collision>
-        <inertial>
-            <origin xyz='0 0 0' rpy='0 0 0'/>
-            <mass value='1'/>
-            <xacro:cylinder_inertia m="1" r="${wheel_base_radius}" h="${wheel_base_length}"/>
+                <cylinder radius='${wheel_radius}' length='${wheel_base_length}'/>
+            </geometry>
+            <material name='gray'>
+                <color rgba='0.5 0.5 0.5 1.0'/>
+            </material>
+        </visual>
+        <collision>
+            <origin xyz='0 0 0' rpy='0 0 0'/>
+            <geometry>
+                <cylinder radius='${wheel_radius}' length='${wheel_base_length}'/>
+            </geometry>
+        </collision>
+        <inertial>
+            <origin xyz='0 0 0' rpy='0 0 0'/>
+            <mass value='1'/>
+            <xacro:cylinder_inertia m="1" r="${wheel_radius}" h="${wheel_base_length}"/>
         </inertial>
     </link>
@@ -424,5 +424,5 @@
         <parent link='wheel_steer_to_wheel'/>
         <child link='wheel'/>
-        <origin xyz='${wheel_steer_to_wheel_length/2+wheel_lenght/2} 0 ${-wheel_steer_to_wheel_height/2}' rpy='0 1.5707 0'/>
+        <origin xyz='${wheel_steer_to_wheel_length/2+wheel_length/2} 0 ${-wheel_steer_to_wheel_height/2}' rpy='0 1.5707 0'/>
         <axis xyz='0 0 1'/>
     </joint>

Commit message: Wheels

File: ros2_ws/src/my_rover/urdf/rover_properties.xacro (robot description, xacro)
@@ -15,5 +15,5 @@
     <xacro:property name='wheel_steer_to_wheel_length' value='0.04'/>
     <xacro:property name='wheel_steer_to_wheel_width' value='0.07'/>
-    <xacro:property name='wheel_steer_to_wheel_height' value='0.15'/>
+    <xacro:property name='wheel_steer_to_wheel_height' value='0.1'/>
     <xacro:property name='wheel_length' value='0.065'/>
     <xacro:property name='wheel_radius' value='${wheel_steer_to_wheel_height*0.9}'/>

Commit message: Wheels

File: ros2_ws/src/my_rover/urdf/rover_properties.xacro (robot description, xacro)
@@ -6,5 +6,5 @@
     <xacro:property name='chassis_suspension_rod_length' value='0.1'/>
     <xacro:property name='chassis_suspension_rod_radius' value='0.02'/>
-    <xacro:property name='suspension_rod_length' value='${sqrt((chassis_length/2)**2 + (chassis_height/2)**2)}'/>
+    <xacro:property name='suspension_rod_length' value='${sqrt((chassis_length/2-wheel_base_radius)**2 + (chassis_height/2-wheel_base_length)**2)}'/>
     <xacro:property name='suspension_rod_radius' value='0.02'/>
     <xacro:property name='wheel_base_length' value='0.065'/>

File: ros2_ws/src/my_rover/urdf/suspension.xacro (robot description, xacro)
@@ -150,20 +150,20 @@
         <parent link='chassis_suspension_rod'/>
         <child link='suspension_rod'/>
-        <origin xyz='0 0 ${-chassis_suspension_rod_length/3}' rpy='${atan2(chassis_height/2 ,chassis_length/2)} ${-pi/2} 0'/>
+        <origin xyz='0 0 ${-chassis_suspension_rod_length/3}' rpy='${atan2((chassis_height/2-wheel_base_lenght) ,(chassis_length/2-wheel_base_radius))} ${-pi/2} 0'/>
     </joint>
     <joint name='suspension_rod_2_joint' type='fixed'>
         <parent link='chassis_suspension_rod_2'/>
         <child link='suspension_rod_2'/>
-        <origin xyz='0 0 ${chassis_suspension_rod_length/3}' rpy='${atan2(chassis_height/2 ,chassis_length/2)} ${-pi/2} 0'/>
+        <origin xyz='0 0 ${chassis_suspension_rod_length/3}' rpy='${atan2((chassis_height/2-wheel_base_lenght) ,(chassis_length/2-wheel_base_radius))} ${-pi/2} 0'/>
     </joint>
     <joint name='suspension_rod_3_joint' type='fixed'>
         <parent link='chassis_suspension_rod'/>
         <child link='suspension_rod_3'/>
-        <origin xyz='0 0 ${-chassis_suspension_rod_length/3}' rpy='${atan2(chassis_height/2 ,chassis_length/2)} ${pi/2} 0'/>
+        <origin xyz='0 0 ${-chassis_suspension_rod_length/3}' rpy='${atan2((chassis_height/2-wheel_base_lenght) ,(chassis_length/2-wheel_base_radius))} ${pi/2} 0'/>
     </joint>
     <joint name='suspension_rod_4_joint' type='fixed'>
         <parent link='chassis_suspension_rod_2'/>
         <child link='suspension_rod_4'/>
-        <origin xyz='0 0 ${chassis_suspension_rod_length/3}' rpy='${atan2(chassis_height/2 ,chassis_length/2)} ${pi/2} 0'/>
+        <origin xyz='0 0 ${chassis_suspension_rod_length/3}' rpy='${atan2((chassis_height/2-wheel_base_lenght) ,(chassis_length/2-wheel_base_radius))} ${pi/2} 0'/>
     </joint>
 </robot>

Commit message: Wheels

File: ros2_ws/src/my_rover/urdf/rover_properties.xacro (robot description, xacro)
@@ -15,5 +15,5 @@
     <xacro:property name='wheel_steer_to_wheel_length' value='0.04'/>
     <xacro:property name='wheel_steer_to_wheel_width' value='0.07'/>
-    <xacro:property name='wheel_steer_to_wheel_height' value='0.1'/>
+    <xacro:property name='wheel_steer_to_wheel_height' value='0.125'/>
     <xacro:property name='wheel_length' value='0.065'/>
     <xacro:property name='wheel_radius' value='${wheel_steer_to_wheel_height*0.9}'/>
