Commit message: Updated sensor placements

File: description/chassis.xacro (robot description, xacro)
@@ -37,24 +37,104 @@
     <origin xyz="0.0 0.0 0.0" rpy="0.0 0.0 0.0"/>
   </joint>
-  <link name="mast_link">
+  <!-- ================= LIDAR MAST & MOUNT ================= -->
+  <link name="lidar_mast_link">
     <visual>
-      <geometry><cylinder radius="0.01" length="0.4"/></geometry>
-      <origin xyz="0.0 0.0 0.2" rpy="0.0 0.0 0.0"/>
-      <material name="white"/>
+      <geometry><cylinder radius="${lidar_mast_radius}" length="${lidar_mast_height}"/></geometry>
+      <material name="black"/>
+      <origin xyz="0 0 ${lidar_mast_height/2}" rpy="0 0 0"/>
     </visual>
     <collision>
-      <geometry><cylinder radius="0.01" length="0.4"/></geometry>
-      <origin xyz="0.0 0.0 0.2" rpy="0.0 0.0 0.0"/>
+      <geometry><cylinder radius="${lidar_mast_radius}" length="${lidar_mast_height}"/></geometry>
+      <origin xyz="0 0 ${lidar_mast_height/2}" rpy="0 0 0"/>
     </collision>
     <inertial>
-      <mass value="0.2"/>
-      <inertia ixx="0.001" ixy="0.0" ixz="0.0" iyy="0.001" iyz="0.0" izz="0.001"/>
+      <mass value="0.5"/>
+      <inertia ixx="0.01" ixy="0" ixz="0" iyy="0.01" iyz="0" izz="0.01"/>
     </inertial>
   </link>
-  <joint name="mast_joint" type="fixed">
+  <joint name="lidar_mast_joint" type="fixed">
     <parent link="base_link"/>
-    <child link="mast_link"/>
-    <origin xyz="${-base_length / 2 + 0.05} 0.1 ${base_height / 2}" rpy="0.0 0.0 0.0"/>
+    <child link="lidar_mast_link"/>
+    <origin xyz="${lidar_mast_x_offset} 0.0 ${base_height/2 + 0.01}" rpy="0 0 0"/>
   </joint>
+  <link name="lidar_plate_link">
+    <visual>
+      <geometry><cylinder radius="0.04" length="0.005"/></geometry>
+      <material name="grey"/>
+    </visual>
+    <collision>
+      <geometry><cylinder radius="0.04" length="0.005"/></geometry>
+    </collision>
+    <inertial>
+      <mass value="0.05"/>
+      <inertia ixx="0.0001" ixy="0" ixz="0" iyy="0.0001" iyz="0" izz="0.0001"/>
+    </inertial>
+  </link>
+  <joint name="lidar_plate_joint" type="fixed">
+    <parent link="lidar_mast_link"/>
+    <child link="lidar_plate_link"/>
+    <origin xyz="0.0 0.0 ${lidar_mast_height + 0.0025}" rpy="0 0 0"/>
+  </joint>
+  <!-- ================= 2D LIDAR ================= -->
+  <link name="lidar_link">
+    <visual>
+      <geometry><cylinder radius="0.05" length="0.04"/></geometry>
+      <material name="black"/>
+    </visual>
+    <collision>
+      <geometry><cylinder radius="0.05" length="0.04"/></geometry>
+    </collision>
+    <inertial>
+      <mass value="0.1"/>
+      <inertia ixx="0.001" ixy="0" ixz="0" iyy="0.001" iyz="0" izz="0.001"/>
+    </inertial>
+  </link>
+  <joint name="lidar_joint" type="fixed">
+    <parent link="lidar_plate_link"/>
+    <child link="lidar_link"/>
+    <origin xyz="0 0 0.0225" rpy="0 0 0"/>
+  </joint>
+  <!-- ================= CAMERA EXTENSION BEAM ================= -->
+  <link name="camera_beam_link">
+    <visual>
+      <geometry><box size="${camera_beam_length} 0.03 0.03"/></geometry>
+      <material name="black"/>
+      <origin xyz="${camera_beam_length/2} 0 0" rpy="0 0 0"/>
+    </visual>
+    <collision>
+      <geometry><box size="${camera_beam_length} 0.03 0.03"/></geometry>
+      <origin xyz="${camera_beam_length/2} 0 0" rpy="0 0 0"/>
+    </collision>
+    <inertial>
+      <mass value="0.3"/>
+      <inertia ixx="0.001" ixy="0" ixz="0" iyy="0.001" iyz="0" izz="0.001"/>
+    </inertial>
+  </link>
+  <joint name="camera_beam_joint" type="fixed">
+    <parent link="base_link"/>
+    <child link="camera_beam_link"/>
+    <origin xyz="${camera_beam_x_start} ${camera_beam_y_offset} ${camera_beam_z_offset}" rpy="0 0 0"/>
+  </joint>
+  <!-- ================= CAMERA MOUNTING PLATE ================= -->
+  <link name="camera_mount_plate">
+    <visual>
+      <geometry><box size="0.01 0.06 0.06"/></geometry>
+      <material name="grey"/>
+    </visual>
+    <collision>
+      <geometry><box size="0.01 0.06 0.06"/></geometry>
+    </collision>
+    <inertial>
+      <mass value="0.05"/>
+      <inertia ixx="0.001" ixy="0" ixz="0" iyy="0.001" iyz="0" izz="0.001"/>
+    </inertial>
+  </link>
+  <joint name="camera_plate_joint" type="fixed">
+    <parent link="camera_beam_link"/>
+    <child link="camera_mount_plate"/>
+    <!-- Attached to the tip of the beam, applying the downward tilt here -->
+    <origin xyz="${camera_beam_length} 0 0" rpy="0 ${camera_pitch} 0"/>
+  </joint>
+  <!-- ================= ZED 2i CAMERA REPLICA ================= -->
   <link name="camera_link">
     <visual>
@@ -62,25 +142,24 @@
       <material name="white"/>
     </visual>
-    <visual>
-      <origin xyz="0.02 0.04 0.0" rpy="0.0 1.5708 0.0"/>
-      <geometry><cylinder radius="0.012" length="0.01"/></geometry>
-      <material name="black"/>
-    </visual>
-    <visual>
-      <origin xyz="0.02 -0.04 0.0" rpy="0.0 1.5708 0.0"/>
-      <geometry><cylinder radius="0.012" length="0.01"/></geometry>
-      <material name="black"/>
-    </visual>
+    <collision>
+      <geometry><box size="0.04 0.14 0.04"/></geometry>
+    </collision>
+    <inertial>
+      <mass value="0.16"/>
+      <inertia ixx="0.001" ixy="0" ixz="0" iyy="0.001" iyz="0" izz="0.001"/>
+    </inertial>
   </link>
   <joint name="camera_joint" type="fixed">
-    <parent link="mast_link"/>
+    <parent link="camera_mount_plate"/>
     <child link="camera_link"/>
-    <origin xyz="0.0 0.0 0.4" rpy="0.0 0.0 0.0"/>
+    <!-- Sits perfectly flush against the tilted plate -->
+    <origin xyz="0.025 0 0" rpy="0 0 0"/>
   </joint>
+  <!-- Optical frame to match ROS image standards -->
   <link name="camera_optical_link"/>
   <joint name="camera_optical_joint" type="fixed">
     <parent link="camera_link"/>
     <child link="camera_optical_link"/>
-    <origin xyz="0.0 0.0 0.0" rpy="-1.5708 0.0 -1.5708"/>
+    <origin xyz="0 0 0" rpy="-1.5708 0 -1.5708"/>
   </joint>
 </robot>

File: description/rover.urdf.xacro (robot description, xacro)
@@ -1,4 +1,4 @@
 <?xml version="1.0"?>
-<robot xmlns:xacro="http://www.ros.org/wiki/xacro" name="ares_nova_v2">
+<robot xmlns:xacro="http://www.ros.org/wiki/xacro" name="autonavtest">
   <!-- INCLUDES -->
   <xacro:include filename="rover_properties.xacro"/>
@@ -57,5 +57,5 @@
   <gazebo>
     <plugin filename="gz_ros2_control-system" name="gz_ros2_control::GazeboSimROS2ControlPlugin">
-      <parameters>$(find ares_nova_v2)/config/ros2_controllers.yaml</parameters>
+      <parameters>$(find autonavtest)/config/ros2_controllers.yaml</parameters>
     </plugin>
   </gazebo>
@@ -69,17 +69,4 @@
   </gazebo>
   <!-- GAZEBO SENSORS -->
-  <gazebo reference="camera_link">
-    <sensor type="camera" name="rover_camera">
-      <always_on>1</always_on>
-      <topic>/camera/image_raw</topic>
-      <update_rate>30.0</update_rate>
-      <visualize>true</visualize>
-      <camera name="head">
-        <horizontal_fov>1.3962634</horizontal_fov>
-        <image><width>800</width><height>800</height><format>R8G8B8</format></image>
-        <clip><near>0.02</near><far>300.0</far></clip>
-      </camera>
-    </sensor>
-  </gazebo>
   <gazebo reference="imu_link">
     <sensor name="rover_imu" type="imu">
@@ -91,3 +78,52 @@
     </sensor>
   </gazebo>
+  <!-- 2D LIDAR SENSOR PLUGIN -->
+  <gazebo reference="lidar_link">
+    <sensor name="lidar" type="gpu_lidar">
+      <always_on>true</always_on>
+      <visualize>true</visualize>
+      <update_rate>10</update_rate>
+      <topic>/scan</topic>
+      <gz_frame_id>lidar_link</gz_frame_id>
+      <lidar>
+        <scan>
+          <horizontal>
+            <samples>360</samples>
+            <resolution>1.0</resolution>
+            <min_angle>-3.14159</min_angle>
+            <max_angle>3.14159</max_angle>
+          </horizontal>
+        </scan>
+        <range>
+          <min>0.15</min>
+          <max>12.0</max>
+          <resolution>0.01</resolution>
+        </range>
+      </lidar>
+    </sensor>
+  </gazebo>
+  <!-- ZED 2i FUNCTIONAL REPLICA (RGB + Depth) -->
+  <gazebo reference="camera_link">
+    <sensor name="depth_camera" type="rgbd_camera">
+      <always_on>true</always_on>
+      <visualize>true</visualize>
+      <update_rate>30.0</update_rate>
+      <topic>/depth_camera/image_raw</topic>
+      <gz_frame_id>camera_link</gz_frame_id>
+      <camera>
+        <!-- ~110 Degree Horizontal FOV to match ZED 2i -->
+        <horizontal_fov>1.92</horizontal_fov>
+        <image>
+          <width>1280</width>
+          <height>720</height>
+          <format>R8G8B8</format>
+        </image>
+        <clip>
+          <!-- ZED 2i realistic depth limits -->
+          <near>0.3</near>
+          <far>20.0</far>
+        </clip>
+      </camera>
+    </sensor>
+  </gazebo>
 </robot>

File: description/rover_properties.xacro (robot description, xacro)
@@ -22,4 +22,16 @@
   <!-- PRESERVED SPACING PADDING -->
   <xacro:property name="susp_dy" value="${(base_width / 2) + 0.08}"/>
+  <!-- LIDAR MAST PARAMETERS -->
+  <xacro:property name="lidar_mast_radius" value="0.015" />
+  <xacro:property name="lidar_mast_height" value="0.325" /> <!-- Halved height -->
+  <xacro:property name="lidar_mast_x_offset" value="-0.15" />
+  <!-- CAMERA EXTENSION BEAM PARAMETERS -->
+  <xacro:property name="camera_beam_y_offset" value="-0.15" />
+  <!-- Start the beam 10cm inside the chassis so it sits on the deck -->
+  <xacro:property name="camera_beam_x_start" value="${base_length/2 - 0.1}" />
+  <!-- Mathematically flush with the top of the gold deck -->
+  <xacro:property name="camera_beam_z_offset" value="${base_height/2 + 0.025}" />
+  <xacro:property name="camera_beam_length" value="0.25" />
+  <xacro:property name="camera_pitch" value="0.26" /> <!-- Tilted downward ~15 degrees -->
   <!-- MATERIALS -->
   <material name="black"><color rgba="0.1 0.1 0.1 1"/></material>

Commit message: Added gps and fixed steer link placement

File: description/chassis.xacro (robot description, xacro)
@@ -5,5 +5,5 @@
     <parent link="base_footprint"/>
     <child link="base_link"/>
-    <origin xyz="0.0 0.0 ${wheel_zoffset}" rpy="0.0 0.0 0.0"/>
+    <origin xyz="0.0 0.0 ${wheel_zoffset + 0.08}" rpy="0.0 0.0 0.0"/>
   </joint>
   <link name="base_link">
@@ -163,3 +163,22 @@
     <origin xyz="0 0 0" rpy="-1.5708 0 -1.5708"/>
   </joint>
+  <!-- ================= GPS MODULE ================= -->
+  <link name="gps_link">
+    <visual>
+      <geometry><box size="0.04 0.04 0.015"/></geometry>
+      <material name="black"/>
+    </visual>
+    <collision>
+      <geometry><box size="0.04 0.04 0.015"/></geometry>
+    </collision>
+    <inertial>
+      <mass value="0.05"/>
+      <inertia ixx="0.0001" ixy="0" ixz="0" iyy="0.0001" iyz="0" izz="0.0001"/>
+    </inertial>
+  </link>
+  <joint name="gps_joint" type="fixed">
+    <parent link="base_link"/>
+    <child link="gps_link"/>
+    <origin xyz="${gps_x_offset} ${gps_y_offset} ${gps_z_offset}" rpy="0 0 0"/>
+  </joint>
 </robot>

File: description/rover.urdf.xacro (robot description, xacro)
@@ -69,4 +69,13 @@
   </gazebo>
   <!-- GAZEBO SENSORS -->
+  <!-- GPS SENSOR PLUGIN -->
+  <gazebo reference="gps_link">
+    <sensor name="rover_gps" type="navsat">
+      <always_on>true</always_on>
+      <update_rate>10.0</update_rate>
+      <topic>/gps/fix</topic>
+      <gz_frame_id>gps_link</gz_frame_id>
+    </sensor>
+  </gazebo>
   <gazebo reference="imu_link">
     <sensor name="rover_imu" type="imu">

File: description/rover_properties.xacro (robot description, xacro)
@@ -34,4 +34,8 @@
   <xacro:property name="camera_beam_length" value="0.25" />
   <xacro:property name="camera_pitch" value="0.26" /> <!-- Tilted downward ~15 degrees -->
+  <!-- GPS MODULE PARAMETERS -->
+  <xacro:property name="gps_x_offset" value="-0.25" /> <!-- Rear edge -->
+  <xacro:property name="gps_y_offset" value="0.25" />  <!-- Left edge -->
+  <xacro:property name="gps_z_offset" value="${base_height/2 + 0.015}" /> <!-- On the gold deck -->
   <!-- MATERIALS -->
   <material name="black"><color rgba="0.1 0.1 0.1 1"/></material>

File: description/wheel.xacro (robot description, xacro)
@@ -39,5 +39,5 @@
       <parent link="${prefix}_steering_link"/>
       <child link="${prefix}_wheel_link"/>
-      <origin xyz="0.0 0.0 -0.1" rpy="-1.5708 0.0 0.0"/>
+      <origin xyz="0.0 0.0 -0.18" rpy="-1.5708 0.0 0.0"/>
       <axis xyz="0 0 1"/>
     </joint>

Commit message: Optimized URDF: added drive motor clearance, removed LiDAR and physical mounts, configured GPS coordinates

File: description/chassis.xacro (robot description, xacro)
@@ -5,5 +5,5 @@
     <parent link="base_footprint"/>
     <child link="base_link"/>
-    <origin xyz="0.0 0.0 ${wheel_zoffset + 0.08}" rpy="0.0 0.0 0.0"/>
+    <origin xyz="0.0 0.0 ${wheel_zoffset + 0.23}" rpy="0.0 0.0 0.0"/>
   </joint>
   <link name="base_link">
@@ -37,104 +37,5 @@
     <origin xyz="0.0 0.0 0.0" rpy="0.0 0.0 0.0"/>
   </joint>
-  <!-- ================= LIDAR MAST & MOUNT ================= -->
-  <link name="lidar_mast_link">
-    <visual>
-      <geometry><cylinder radius="${lidar_mast_radius}" length="${lidar_mast_height}"/></geometry>
-      <material name="black"/>
-      <origin xyz="0 0 ${lidar_mast_height/2}" rpy="0 0 0"/>
-    </visual>
-    <collision>
-      <geometry><cylinder radius="${lidar_mast_radius}" length="${lidar_mast_height}"/></geometry>
-      <origin xyz="0 0 ${lidar_mast_height/2}" rpy="0 0 0"/>
-    </collision>
-    <inertial>
-      <mass value="0.5"/>
-      <inertia ixx="0.01" ixy="0" ixz="0" iyy="0.01" iyz="0" izz="0.01"/>
-    </inertial>
-  </link>
-  <joint name="lidar_mast_joint" type="fixed">
-    <parent link="base_link"/>
-    <child link="lidar_mast_link"/>
-    <origin xyz="${lidar_mast_x_offset} 0.0 ${base_height/2 + 0.01}" rpy="0 0 0"/>
-  </joint>
-  <link name="lidar_plate_link">
-    <visual>
-      <geometry><cylinder radius="0.04" length="0.005"/></geometry>
-      <material name="grey"/>
-    </visual>
-    <collision>
-      <geometry><cylinder radius="0.04" length="0.005"/></geometry>
-    </collision>
-    <inertial>
-      <mass value="0.05"/>
-      <inertia ixx="0.0001" ixy="0" ixz="0" iyy="0.0001" iyz="0" izz="0.0001"/>
-    </inertial>
-  </link>
-  <joint name="lidar_plate_joint" type="fixed">
-    <parent link="lidar_mast_link"/>
-    <child link="lidar_plate_link"/>
-    <origin xyz="0.0 0.0 ${lidar_mast_height + 0.0025}" rpy="0 0 0"/>
-  </joint>
-  <!-- ================= 2D LIDAR ================= -->
-  <link name="lidar_link">
-    <visual>
-      <geometry><cylinder radius="0.05" length="0.04"/></geometry>
-      <material name="black"/>
-    </visual>
-    <collision>
-      <geometry><cylinder radius="0.05" length="0.04"/></geometry>
-    </collision>
-    <inertial>
-      <mass value="0.1"/>
-      <inertia ixx="0.001" ixy="0" ixz="0" iyy="0.001" iyz="0" izz="0.001"/>
-    </inertial>
-  </link>
-  <joint name="lidar_joint" type="fixed">
-    <parent link="lidar_plate_link"/>
-    <child link="lidar_link"/>
-    <origin xyz="0 0 0.0225" rpy="0 0 0"/>
-  </joint>
-  <!-- ================= CAMERA EXTENSION BEAM ================= -->
-  <link name="camera_beam_link">
-    <visual>
-      <geometry><box size="${camera_beam_length} 0.03 0.03"/></geometry>
-      <material name="black"/>
-      <origin xyz="${camera_beam_length/2} 0 0" rpy="0 0 0"/>
-    </visual>
-    <collision>
-      <geometry><box size="${camera_beam_length} 0.03 0.03"/></geometry>
-      <origin xyz="${camera_beam_length/2} 0 0" rpy="0 0 0"/>
-    </collision>
-    <inertial>
-      <mass value="0.3"/>
-      <inertia ixx="0.001" ixy="0" ixz="0" iyy="0.001" iyz="0" izz="0.001"/>
-    </inertial>
-  </link>
-  <joint name="camera_beam_joint" type="fixed">
-    <parent link="base_link"/>
-    <child link="camera_beam_link"/>
-    <origin xyz="${camera_beam_x_start} ${camera_beam_y_offset} ${camera_beam_z_offset}" rpy="0 0 0"/>
-  </joint>
-  <!-- ================= CAMERA MOUNTING PLATE ================= -->
-  <link name="camera_mount_plate">
-    <visual>
-      <geometry><box size="0.01 0.06 0.06"/></geometry>
-      <material name="grey"/>
-    </visual>
-    <collision>
-      <geometry><box size="0.01 0.06 0.06"/></geometry>
-    </collision>
-    <inertial>
-      <mass value="0.05"/>
-      <inertia ixx="0.001" ixy="0" ixz="0" iyy="0.001" iyz="0" izz="0.001"/>
-    </inertial>
-  </link>
-  <joint name="camera_plate_joint" type="fixed">
-    <parent link="camera_beam_link"/>
-    <child link="camera_mount_plate"/>
-    <!-- Attached to the tip of the beam, applying the downward tilt here -->
-    <origin xyz="${camera_beam_length} 0 0" rpy="0 ${camera_pitch} 0"/>
-  </joint>
-  <!-- ================= ZED 2i CAMERA REPLICA ================= -->
+  <!-- ================= ZED 2i CAMERA (FLOATING) ================= -->
   <link name="camera_link">
     <visual>
@@ -151,8 +52,8 @@
   </link>
   <joint name="camera_joint" type="fixed">
-    <parent link="camera_mount_plate"/>
+    <parent link="base_link"/>
     <child link="camera_link"/>
-    <!-- Sits perfectly flush against the tilted plate -->
-    <origin xyz="0.025 0 0" rpy="0 0 0"/>
+    <!-- Floating exactly where the extension beam used to end -->
+    <origin xyz="${camera_beam_x_start + camera_beam_length} ${camera_beam_y_offset} ${camera_beam_z_offset}" rpy="0 ${camera_pitch} 0"/>
   </joint>
   <!-- Optical frame to match ROS image standards -->
@@ -163,5 +64,5 @@
     <origin xyz="0 0 0" rpy="-1.5708 0 -1.5708"/>
   </joint>
-  <!-- ================= GPS MODULE ================= -->
+  <!-- ================= GPS MODULE (FLOATING) ================= -->
   <link name="gps_link">
     <visual>
@@ -180,4 +81,5 @@
     <parent link="base_link"/>
     <child link="gps_link"/>
+    <!-- Floating on the rear-left corner -->
     <origin xyz="${gps_x_offset} ${gps_y_offset} ${gps_z_offset}" rpy="0 0 0"/>
   </joint>

File: description/rover.urdf.xacro (robot description, xacro)
@@ -87,29 +87,4 @@
     </sensor>
   </gazebo>
-  <!-- 2D LIDAR SENSOR PLUGIN -->
-  <gazebo reference="lidar_link">
-    <sensor name="lidar" type="gpu_lidar">
-      <always_on>true</always_on>
-      <visualize>true</visualize>
-      <update_rate>10</update_rate>
-      <topic>/scan</topic>
-      <gz_frame_id>lidar_link</gz_frame_id>
-      <lidar>
-        <scan>
-          <horizontal>
-            <samples>360</samples>
-            <resolution>1.0</resolution>
-            <min_angle>-3.14159</min_angle>
-            <max_angle>3.14159</max_angle>
-          </horizontal>
-        </scan>
-        <range>
-          <min>0.15</min>
-          <max>12.0</max>
-          <resolution>0.01</resolution>
-        </range>
-      </lidar>
-    </sensor>
-  </gazebo>
   <!-- ZED 2i FUNCTIONAL REPLICA (RGB + Depth) -->
   <gazebo reference="camera_link">

File: description/wheel.xacro (robot description, xacro)
@@ -15,4 +15,5 @@
       <parent link="${parent_arm}"/>
       <child link="${prefix}_steering_link"/>
+      <!-- Removed the gap here so the steering motor sits perfectly flush with the suspension arm -->
       <origin xyz="${(suspension_length / 2) * x_reflect + steer_xoffset} 0.0 ${steer_zoffset}" rpy="0.0 0.0 0.0"/>
       <axis xyz="0 0 1"/>
@@ -39,5 +40,6 @@
       <parent link="${prefix}_steering_link"/>
       <child link="${prefix}_wheel_link"/>
-      <origin xyz="0.0 0.0 -0.18" rpy="-1.5708 0.0 0.0"/>
+      <!-- Added the 0.15m gap HERE, below the motor block, pushing the wheel down (-0.18 - 0.15 = -0.33) -->
+      <origin xyz="0.0 0.0 -0.33" rpy="-1.5708 0.0 0.0"/>
       <axis xyz="0 0 1"/>
     </joint>
