Commit message: pitch

File: ros_ws/src/description/rover_properties.xacro (robot description, xacro)
@@ -33,5 +33,5 @@
   <xacro:property name="camera_beam_z_offset" value="${base_height/2 + 0.025}" />
   <xacro:property name="camera_beam_length" value="0.25" />
-  <xacro:property name="camera_pitch" value="0.26" /> <!-- Tilted downward ~15 degrees -->
+  <xacro:property name="camera_pitch" value="0.0" />
   <!-- GPS MODULE PARAMETERS -->
   <xacro:property name="gps_x_offset" value="-0.25" /> <!-- Rear edge -->
