Commit message: pitch

File: ros_ws/src/description/rover.urdf.xacro (robot description, xacro)
@@ -85,7 +85,7 @@
     <update_rate>15.0</update_rate>
     <topic>/depth_camera/image_raw</topic>
-    <ignition_frame_id>camera_optical_link</ignition_frame_id>
-    <gz_frame_id>camera_optical_link</gz_frame_id>
+    <gz_frame_id>camera_link</gz_frame_id>
     <camera>
+      <optical_frame_id>camera_optical_link</optical_frame_id>
       <horizontal_fov>1.92</horizontal_fov>
       <image><width>640</width><height>480</height><format>R8G8B8</format></image>

File: ros_ws/src/description/rover_properties.xacro (robot description, xacro)
@@ -33,5 +33,5 @@
   <xacro:property name="camera_beam_z_offset" value="${base_height/2 + 0.025}" />
   <xacro:property name="camera_beam_length" value="0.25" />
-  <xacro:property name="camera_pitch" value="0.0" />
+  <xacro:property name="camera_pitch" value="0.26" /> <!-- Tilted downward ~15 degrees -->
   <!-- GPS MODULE PARAMETERS -->
   <xacro:property name="gps_x_offset" value="-0.25" /> <!-- Rear edge -->
