Commit message: Updated

File: ros_ws/src/description/chassis.xacro (robot description, xacro)
@@ -55,5 +55,5 @@
     <child link="camera_link"/>
     <!-- Floating exactly where the extension beam used to end -->
-    <origin xyz="${camera_beam_x_start + camera_beam_length} ${camera_beam_y_offset} ${camera_beam_z_offset}" rpy="0 ${camera_pitch} 0"/>
+    <origin xyz="${camera_beam_x_start + camera_beam_length} ${camera_beam_y_offset} ${camera_beam_z_offset}" rpy="0 0 0"/>
   </joint>
   <!-- Optical frame to match ROS image standards -->
@@ -62,5 +62,5 @@
     <parent link="camera_link"/>
     <child link="camera_optical_link"/>
-    <origin xyz="0 0 0" rpy="-1.5708 0 -1.5708"/>
+    <origin xyz="0 0 0" rpy="-1.1781 0 -1.5708"/>
   </joint>
   <!-- ================= GPS MODULE (FLOATING) ================= -->

File: ros_ws/src/description/rover.urdf.xacro (robot description, xacro)
@@ -55,8 +55,7 @@
     </joint>
   </ros2_control>
-  <xacro:arg name="params_file" default="$(find autonavtest)/config/ros2_controllers.yaml"/>
   <gazebo>
     <plugin filename="gz_ros2_control-system" name="gz_ros2_control::GazeboSimROS2ControlPlugin">
-      <parameters>$(arg params_file)</parameters>
+      <parameters>$(find autonavtest)/config/ros2_controllers.yaml</parameters>
     </plugin>
   </gazebo>
@@ -85,7 +84,7 @@
     <update_rate>15.0</update_rate>
     <topic>/depth_camera/image_raw</topic>
-    <gz_frame_id>camera_link</gz_frame_id>
+    <ignition_frame_id>camera_optical_link</ignition_frame_id>
+    <gz_frame_id>camera_optical_link</gz_frame_id>
     <camera>
-      <optical_frame_id>camera_optical_link</optical_frame_id>
       <horizontal_fov>1.92</horizontal_fov>
       <image><width>640</width><height>480</height><format>R8G8B8</format></image>

Commit message: errors

File: ros_ws/src/description/chassis.xacro (robot description, xacro)
@@ -55,5 +55,6 @@
     <child link="camera_link"/>
     <!-- Floating exactly where the extension beam used to end -->
-    <origin xyz="${camera_beam_x_start + camera_beam_length} ${camera_beam_y_offset} ${camera_beam_z_offset}" rpy="0 0 0"/>
+    <!-- Apply the physical downward pitch to the camera mount. -->
+    <origin xyz="${camera_beam_x_start + camera_beam_length} ${camera_beam_y_offset} ${camera_beam_z_offset}" rpy="0 ${camera_pitch} 0"/>
   </joint>
   <!-- Optical frame to match ROS image standards -->
@@ -62,5 +63,6 @@
     <parent link="camera_link"/>
     <child link="camera_optical_link"/>
-    <origin xyz="0 0 0" rpy="-1.1781 0 -1.5708"/>
+    <!-- REP-103 camera-link -> optical-frame rotation (Z forward, X right). -->
+    <origin xyz="0 0 0" rpy="-1.5708 0 -1.5708"/>
   </joint>
   <!-- ================= GPS MODULE (FLOATING) ================= -->
